File: lm3410-sepic/lm3410-sepic-led-driver-16mm-mk-4.brd (EAGLE design)
At the start: 16 x 16 mm, 13 parts

Commit message: helps if i add the damn files
Parts:
- +: value M01PTH-KIT -> M01PTH-1.2MM; device A_butts:1X01-KIT -> A_butts:1X01-1.2MM
- -: value M01NOSILK-KIT -> M01PTH-1.2MM-NS; device A_butts:1X01NS-KIT -> A_butts:1X01-1.2MM-NS
- D1: value BAT20J -> MBRA140; device A_butts:SOD-323 -> A_butts:SMA-DIODE
- L1, L2: device A_butts:INDUCTOR_2X1.6MM -> A_butts:TAIYO-YUDEN-30XX
- LM3410: value LM3410XMYA -> LM3410XMF; device A_butts:SOP65P490X110-9N-A -> A_butts:SOT95P285X120-5N
- moved JBATT- 11.0 mm to (13.5, 10.7)
- moved C1 8.01 mm to (9.02, 3.20), turned to 270 degrees
- moved JBATT+ 6.26 mm to (8.00, 5.40)
- moved R1 6.15 mm to (3.70, 7.90), turned to 0 degrees
- moved R2 4.98 mm to (6.98, 3.20), turned to 90 degrees
- moved C2 2.62 mm to (10.5, 7.10), turned to 90 degrees
- moved D1 1.60 mm to (13.2, 7.25), turned to 270 degrees
- moved L1 1.41 mm to (5.05, 10.9), turned to 90 degrees
- moved L2 1.41 mm to (10.9, 10.9), turned to 90 degrees
- moved C3 0.70 mm to (8.00, 12.2)
- moved LM3410 0.20 mm to (8.00, 7.80), turned to 270 degrees
- turned + to 90 degrees
Connections:
- net GND: now also L2.2; no longer L2.P$2, LM3410.6, LM3410.9
- net LED_ANODE: now also +.P$1; no longer +.1
- net LED_CATHODE: now also -.P$1, LM3410.3; no longer -.1, LM3410.5
- net N$1: now also L2.1; no longer L2.P$1
- net SW: now also L1.2, LM3410.1; no longer L1.P$2, LM3410.7
- net VCC: now also L1.1, LM3410.5; no longer L1.P$1, LM3410.3
Routing:
- net SW: track 8.69 -> 6.52 mm
- net N$3: track 1.94 -> 2.55 mm
- net VCC: track 13.7 -> 13.2 mm, vias 0 -> 1
Other:
- board text added: "Septic SEPIC 16mm Rev 4.0 CC-BY-SA-4.0"
- board text removed: "Septic SEPIC 16mm Rev 3.0 CC-BY-SA-4.0"
