File: lm3410-sepic/lm3410-boost-flashlight-driver-17mm-mk-1.1.0.sch (EAGLE design)
At the start: 16 parts, among them Q1 PSMN2R4-30MLD, U1 ATTINY13a, U2 PAM2803

Commit message: bunch of new board word
Parts:
- removed +, -: M01NOT-A-VIA-NOPE, a_parts:M01NOT-A-VIA-NOPE
- removed A, K: M01PTH-1MM-CIR-NS, a_parts:M01PTH-1MM-CIR-NS
- removed Q1: PSMN2R4-30MLD, a_parts:MOSFET-NCHANNELLFPAK33
- removed R1: 0R1, a_parts:RESISTORR0603-TIGHTER
- removed R2: 150K, a_parts:RESISTORR0603-TIGHTER
- removed R3: 33K, a_parts:RESISTORR0603-TIGHTER
- added D2: BAT60A, a_parts:DIODE-SCHOTTKYSOD323
- added LED+, LED-: M01PTH-1MM-CIR-NS, a_parts:M01PTH-1MM-CIR-NS
- C1: value 10uF -> 10u
- C2: value 22uF -> 10u
- D1: value BAT60 -> BAT60A
- FRAME1: VERSION v1.1 -> v1.2
- L1: value 2.2uF -> 10uH
- R4: value 33R -> X; device a_parts:RESISTORR0603-TIGHTER -> a_parts:RESISTORR0805-TIGHTER
- U1: value ATTINY13a -> Tiny25; device a_parts:ATTINY13SOIC-NARROWER -> a_parts:ATTINY45TINY25-SOICN-NARROWER
- U2: value PAM2803 -> LM3410XSDNGG; device a_parts:PAM2803SOT23-6 -> a_parts:LM3410XSDNGG
Connections:
- removed net !SHDN: U1.PB3(ADC3), U2.!SHDN
- removed net GATE: Q1.G, R3.2, R4.2
- removed net LED-: K.1, Q1.D
- new net VCC: D1.C, U1.VCC
- net FB: now also LED-.1, R4.2; no longer Q1.S, R1.2, R3.1
- net GND: now also R4.1, U2.AGND, U2.EPAD, U2.PGND; no longer -.1, R1.1, R2.1, U2.GND
- net LED+: now also D2.C, LED+.1; no longer A.1, D1.C, U2.VO
- net PWM: now also U2.DIM; no longer R4.1
- net SW: now also D2.A, L1.2; no longer D1.A, L1.1
- net VBAT: now also D1.A, L1.1; no longer +.1, L1.2, R2.2, U1.VCC
Other:
- note added: "190mV R4 = ----- I 10mA => 19R 21mA => 9R0 40mA => 4R7 70mA => 2R7 190mA => 1R0 340mA => R560 400mA => R470 950mA => R200 1000mA => R190 1500mA => R130 1900mA => R100"
- note removed: "0.095V Iout = ------ R1"
- note removed: "0R27 = 352 mA 0R22 = 432 mA 0R20 = 475 mA 0R18 = 528 mA 0R15 = 633 mA 0R12 = 792 mA 0R10 = 950 mA"
- moved on the sheet: C1, C2, D1, L1, R4, U1
