File: amc7135/fabflash-mk-2-booster.sch (EAGLE design)
At the start: 15 parts, among them U1 LM2735YMF

Commit message: faaaabulous flashlight in progress
Parts:
- removed C2, C4: (no value), A_butts:CAPACITOR-CERAMICC0805
- removed JP2: M01NOT-A-VIA-NOPE, A_butts:M01NOT-A-VIA-NOPE
- added 5V: M01PTH-1.2MM, A_butts:M01PTH-1.2MM
- added BATT-: M01NOT-A-VIA-NOPE, A_butts:M01NOT-A-VIA-NOPE
- C1: value (none) -> 22uF
- C3: value (none) -> 10uF
- C5: value (none) -> 2.2nF
- C6: value (none) -> 2.2uF
- L1, L2: device A_butts:INDUCTORTAIYO-YUDEN-30XX -> A_butts:INDUCTORTAIYO-YUDEN-40XX
- R1: value (none) -> 10k
- R2: value (none) -> 30k
- R3: value (none) -> 100k
- renumbered JP1 to BATT+
Connections:
- net GND: now also BATT-.1, R1.1; no longer C4.2, R3.1
- net N$2: now also R3.2; no longer R1.1
- net N$8: now also R1.2; no longer R3.2
- net VIN: now also R3.1; no longer C2.1, R1.2
- net VOUT: now also 5V.1; no longer C4.1, JP2.1
Other:
- moved on the sheet: C1, R1, R3
