File: amc7135/fabflash-mk-2.2-driver.sch (EAGLE design)
At the start: 17 parts, among them Q1 MOSFET-PCHANNELIRLML2244, U1 LM2735YMF

Commit message: two new tries at this, about to go for 3
Parts:
- removed BATT+, BATT-: M01NOT-A-VIA-NOPE, A_butts:M01NOT-A-VIA-NOPE
- removed C3: 10uF, A_butts:CAPACITOR-CERAMICC0805
- removed C5: 2.2nF, A_butts:CAPACITOR-CERAMICC0603
- removed C6: 2.2uF, A_butts:CAPACITOR-CERAMICC0805
- removed D1: B340A, A_butts:DIODE-SCHOTTKYB340A
- removed D2: 10V, A_butts:DIODE-ZENERSOD123
- removed L1, L2: 6.8uH, A_butts:INDUCTORTAIYO-YUDEN-40XX
- removed Q1: MOSFET-PCHANNELIRLML2244, A_butts:MOSFET-PCHANNELIRLML2244
- removed R2: 30k, A_butts:RESISTORR0603
- removed R3, R4: 100k, A_butts:RESISTORR0603
- added +, B-, G-, R-, W-: M01SMD_2X3MM, A_butts:M01SMD_2X3MM
- added GND: M01NOT-A-VIA-NOPE, A_butts:M01NOT-A-VIA-NOPE
- added U2, U3, U4, U5: AMC7135SOT-89, A_butts:AMC7135SOT-89
- 5V: value M01PTH-1.2MM -> M01SMD_2X3MM; device A_butts:M01PTH-1.2MM -> A_butts:M01SMD_2X3MM
- C1: value 22uF -> 10uF
- R1: value 10k -> 100k
- U1: value LM2735YMF -> ATTINY84; device A_butts:LM2735YMF -> A_butts:ATTINY84ATTINY84-20MU
Connections:
- removed net BATT+: BATT+.1, Q1.D
- removed net N$2: R3.2, U1.EN
- removed net N$4: D2.A, Q1.G, R4.2
- removed net N$6: C6.2, D1.A, L2.1
- removed net N$8: C5.2, R1.2, R2.1, U1.FB
- removed net VIN: C1.1, D2.C, L1.1, Q1.S, R3.1, U1.VIN
- removed net VOUT: 5V.1, C3.1, C5.1, D1.C, R2.2
- new net 5V: +.1, 5V.1, C1.1, R1.1, U1.VCC
- new net BLUE-: B-.1, U4.LED
- new net BLUEPWM: U1.(PCINT10/INT0/OC0A/CKOUT)PB2, U4.VDD
- new net GREEN-: G-.1, U3.LED
- new net GREENPWM: U1.(PCINT6/OC1A/SDA/MOSI/ADC6)PA6, U3.VDD
- new net RED-: R-.1, U2.LED
- new net REDPWM: U1.(PCINT7/ICP/OC0B/ADC7)PA7, U2.VDD
- new net WHITE-: U5.LED, W-.1
- new net WHITEPWM: U1.(PCINT5/OC1B/MISO/DO/ADC5)PA5, U5.VDD
- net GND: now also GND.1, U2.GND, U3.GND, U4.GND, U5.GND; no longer BATT-.1, C3.2, L2.2, R1.1, R4.1
- net N$1: now also R1.2, U1.(PCINT11/~RESET/DW)PB3; no longer C6.1, L1.2, U1.SW
Other:
- moved on the sheet: 5V, C1, R1
