File: amc7135/fabflash-mk-2.3-booster.sch (EAGLE design)
At the start: 18 parts, among them Q1 MOSFET-PCHANNELIRLML2244, U1 LM2735YMF

Commit message: slowly making progress toward a buildable device
Parts:
- removed BATT-: M01NOT-A-VIA-NOPE, A_butts:M01NOT-A-VIA-NOPE
- added JP4, JP5, JP6: M01PTH-0.9MM-NS, A_butts:M01PTH-0.9MM-NS
- added JP7, JP8: (no value), A_butts:M05SMD-SHORT-2MM
- D1: device A_butts:DIODE-SCHOTTKYB340A -> A_butts:DIODE-SCHOTTKYSOD123
- JP1, JP2: value M01PTH -> M01PTH-0.9MM-NS; device A_butts:M01PTH -> A_butts:M01PTH-0.9MM-NS
- JP3: value M03PTH -> M01PTH-0.9MM-NS; device A_butts:M03PTH -> A_butts:M01PTH-0.9MM-NS
Connections:
- removed net N$3: JP3.1, JP3.2, JP3.3, Q1.D
- new net BATT+: JP7.2, JP7.3, JP7.4, JP8.2, JP8.3, JP8.4, Q1.D
- net 5V: now also JP6.1; no longer JP1.1
- net GND: now also JP3.1, JP7.1, JP7.5, JP8.1, JP8.5; no longer BATT-.1, JP2.1
Other:
- moved on the sheet: JP1, JP2
Changed lines of the file:
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@@
 <setting verticaltext="up"/>
 </settings>
-<grid distance="100" unitdist="mil" unit="mil" style="lines" multiple="1" display="yes" altdistance="1" altunitdist="mil" altunit="mil"/>
+<grid distance="100" unitdist="mil" unit="mil" style="lines" multiple="1" display="yes" altdistance="1" altunitdist="mm" altunit="mm"/>
 <layers>
 <layer number="1" name="Top" color="4" fill="1" visible="yes" active="no"/>
@@
 <part name="C6" library="A_butts" deviceset="CAPACITOR-CERAMIC" device="C0805" value="2.2uF"/>
 <part name="R2" library="A_butts" deviceset="RESISTOR" device="R0603" value="30k"/>
-<part name="D1" library="A_butts" deviceset="DIODE-SCHOTTKY" device="B340A" value="B340A"/>
+<part name="D1" library="A_butts" deviceset="DIODE-SCHOTTKY" device="SOD123" value="B340A"/>
 <part name="L1" library="A_butts" deviceset="INDUCTOR" device="TAIYO-YUDEN-40XX" value="6.8uH"/>
 <part name="L2" library="A_butts" deviceset="INDUCTOR" device="TAIYO-YUDEN-40XX" value="6.8uH"/>
-<part name="BATT-" library="A_butts" deviceset="M01" device="NOT-A-VIA-NOPE"/>
 <part name="R1" library="A_butts" deviceset="RESISTOR" device="R0603" value="10k"/>
 <part name="R3" library="A_butts" deviceset="RESISTOR" device="R0603" value="100k"/>
@@
 <part name="R4" library="A_butts" deviceset="RESISTOR" device="R0603" value="100k"/>
 <part name="GND2" library="A_butts" deviceset="GND" device=""/>
-<part name="JP3" library="A_butts" deviceset="M03" device="PTH" value="M03PTH"/>
-<part name="JP1" library="A_butts" deviceset="M01" device="PTH"/>
-<part name="JP2" library="A_butts" deviceset="M01" device="PTH"/>
+<part name="JP1" library="A_butts" deviceset="M01" device="PTH-0.9MM-NS"/>
+<part name="JP2" library="A_butts" deviceset="M01" device="PTH-0.9MM-NS"/>
+<part name="JP3" library="A_butts" deviceset="M01" device="PTH-0.9MM-NS"/>
+<part name="JP4" library="A_butts" deviceset="M01" device="PTH-0.9MM-NS"/>
+<part name="JP5" library="A_butts" deviceset="M01" device="PTH-0.9MM-NS"/>
+<part name="JP6" library="A_butts" deviceset="M01" device="PTH-0.9MM-NS"/>
+<part name="JP7" library="A_butts" deviceset="M05" device="SMD-SHORT-2MM"/>
+<part name="GND3" library="A_butts" deviceset="GND" device=""/>
+<part name="JP8" library="A_butts" deviceset="M05" device="SMD-SHORT-2MM"/>
+<part name="GND5" library="A_butts" deviceset="GND" device=""/>
 </parts>
 <sheets>
@@
 <instance part="L1" gate="G$1" x="68.58" y="60.96" rot="R90"/>
 <instance part="L2" gate="G$1" x="104.14" y="50.8"/>
-<instance part="BATT-" gate="G$1" x="2.54" y="27.94"/>
 <instance part="R1" gate="G$1" x="119.38" y="35.56" rot="R90"/>
 <instance part="R3" gate="G$1" x="43.18" y="50.8" rot="R270"/>
@@
 <instance part="D2" gate="G$1" x="22.86" y="50.8"/>
 <instance part="R4" gate="G$1" x="17.78" y="38.1" rot="R90"/>
-<instance part="GND2" gate="1" x="73.66" y="78.74"/>
-<instance part="JP3" gate="G$1" x="0" y="60.96"/>
-<instance part="JP1" gate="G$1" x="63.5" y="93.98"/>
-<instance part="JP2" gate="G$1" x="63.5" y="83.82"/>
+<instance part="GND2" gate="1" x="12.7" y="86.36" rot="R90"/>
+<instance part="JP1" gate="G$1" x="-20.32" y="106.68"/>
+<instance part="JP2" gate="G$1" x="-20.32" y="96.52"/>
+<instance part="JP3" gate="G$1" x="-20.32" y="86.36"/>
+<instance part="JP4" gate="G$1" x="-20.32" y="76.2"/>
+<instance part="JP5" gate="G$1" x="-20.32" y="66.04"/>
+<instance part="JP6" gate="G$1" x="-20.32" y="55.88"/>
+<instance part="JP7" gate="G$1" x="0" y="60.96"/>
+<instance part="GND3" gate="1" x="5.08" y="48.26" rot="MR90"/>
+<instance part="JP8" gate="G$1" x="0" y="35.56"/>
+<instance part="GND5" gate="1" x="7.62" y="25.4"/>
 </instances>
 <busses>
@@
 <junction x="119.38" y="27.94"/>
 <label x="27.94" y="25.4" size="1.27" layer="95"/>
-<pinref part="BATT-" gate="G$1" pin="1"/>
-<wire x1="10.16" y1="27.94" x2="17.78" y2="27.94" width="0.1524" layer="91"/>
 <junction x="35.56" y="27.94"/>
 <pinref part="R1" gate="G$1" pin="1"/>
@@
 <wire x1="17.78" y1="27.94" x2="35.56" y2="27.94" width="0.1524" layer="91"/>
 <wire x1="17.78" y1="33.02" x2="17.78" y2="27.94" width="0.1524" layer="91"/>
-<junction x="17.78" y="27.94"/>
-</segment>
-<segment>
-<wire x1="71.12" y1="83.82" x2="73.66" y2="83.82" width="0.1524" layer="91"/>
+</segment>
+<segment>
+<wire x1="-12.7" y1="86.36" x2="7.62" y2="86.36" width="0.1524" layer="91"/>
 <pinref part="GND2" gate="1" pin="GND"/>
-<wire x1="73.66" y1="83.82" x2="73.66" y2="81.28" width="0.1524" layer="91"/>
-<pinref part="JP2" gate="G$1" pin="1"/>
+<pinref part="JP3" gate="G$1" pin="1"/>
+<pinref part="JP7" gate="G$1" pin="5"/>
+<wire x1="7.62" y1="86.36" x2="10.16" y2="86.36" width="0.1524" layer="91"/>
+<wire x1="7.62" y1="66.04" x2="7.62" y2="86.36" width="0.1524" layer="91"/>
+<junction x="7.62" y="86.36"/>
+</segment>
+<segment>
+<pinref part="GND3" gate="1" pin="GND"/>
+<pinref part="JP7" gate="G$1" pin="1"/>
+<wire x1="7.62" y1="48.26" x2="7.62" y2="55.88" width="0.1524" layer="91"/>
+<pinref part="JP8" gate="G$1" pin="5"/>
+<wire x1="7.62" y1="40.64" x2="7.62" y2="48.26" width="0.1524" layer="91"/>
+<junction x="7.62" y="48.26"/>
+</segment>
+<segment>
+<pinref part="JP8" gate="G$1" pin="1"/>
+<pinref part="GND5" gate="1" pin="GND"/>
+<wire x1="7.62" y1="30.48" x2="7.62" y2="27.94" width="0.1524" layer="91"/>
 </segment>
 </net>
@@
 <net name="5V" class="0">
 <segment>
-<wire x1="71.12" y1="93.98" x2="76.2" y2="93.98" width="0.1524" layer="91"/>
-<label x="76.2" y="93.98" size="1.27" layer="95" xref="yes"/>
-<pinref part="JP1" gate="G$1" pin="1"/>
+<wire x1="-12.7" y1="55.88" x2="-10.16" y2="55.88" width="0.1524" layer="91"/>
+<label x="-10.16" y="55.88" size="1.27" layer="95" xref="yes"/>
+<pinref part="JP6" gate="G$1" pin="1"/>
 </segment>
 <segment>
@@
 </segment>
 </net>
-<net name="N$3" class="0">
+<net name="BATT+" class="0">
 <segment>
 <pinref part="Q1" gate="G$1" pin="D"/>
 <wire x1="7.62" y1="60.96" x2="10.16" y2="60.96" width="0.1524" layer="91"/>
-<pinref part="JP3" gate="G$1" pin="2"/>
-<pinref part="JP3" gate="G$1" pin="3"/>
 <wire x1="10.16" y1="60.96" x2="12.7" y2="60.96" width="0.1524" layer="91"/>
 <wire x1="7.62" y1="63.5" x2="10.16" y2="63.5" width="0.1524" layer="91"/>
 <wire x1="10.16" y1="63.5" x2="10.16" y2="60.96" width="0.1524" layer="91"/>
 <junction x="10.16" y="60.96"/>
-<pinref part="JP3" gate="G$1" pin="1"/>
 <wire x1="7.62" y1="58.42" x2="10.16" y2="58.42" width="0.1524" layer="91"/>
 <wire x1="10.16" y1="58.42" x2="10.16" y2="60.96" width="0.1524" layer="91"/>
-</segment>
-</net>
+<pinref part="JP7" gate="G$1" pin="2"/>
+<pinref part="JP7" gate="G$1" pin="3"/>
+<pinref part="JP7" gate="G$1" pin="4"/>
+<wire x1="10.16" y1="58.42" x2="10.16" y2="38.1" width="0.1524" layer="91"/>
+<junction x="10.16" y="58.42"/>
+<pinref part="JP8" gate="G$1" pin="4"/>
+<wire x1="10.16" y1="38.1" x2="7.62" y2="38.1" width="0.1524" layer="91"/>
+<wire x1="10.16" y1="38.1" x2="10.16" y2="35.56" width="0.1524" layer="91"/>
+<junction x="10.16" y="38.1"/>
+<pinref part="JP8" gate="G$1" pin="2"/>
+<wire x1="10.16" y1="35.56" x2="10.16" y2="33.02" width="0.1524" layer="91"/>
+<wire x1="10.16" y1="33.02" x2="7.62" y2="33.02" width="0.1524" layer="91"/>
+<pinref part="JP8" gate="G$1" pin="3"/>
+<wire x1="7.62" y1="35.56" x2="10.16" y2="35.56" width="0.1524" layer="91"/>
+<junction x="10.16" y="35.56"/>
+</segment>
+</net>
