File: amc7135/amc7135-testboard-mk-1.1.sch (EAGLE design)
At the start: 12 parts, among them IC1 ATTiny13, IC2 AMC7135

Commit message: whoa nelly lots of boards never quite finished
Parts:
- AVR_ISP: value AVR_SPI_PRG_6PTH -> AVR_SPI_PRG_6SMD_TEST_POINTS; device A_butts:AVR_SPI_PRG_6PTH -> a_parts:AVR_SPI_PRG_6SMD_TEST_POINTS
- C1: device A_butts:CAPACITOR-CERAMICC0805 -> a_parts:CAPACITOR-CERAMICC0603-TIGHTER
- C2: device A_butts:CAPACITOR-CERAMICC0805 -> a_parts:CAPACITOR-CERAMICC1210
- D1: device A_butts:DIODE-SCHOTTKYSMA -> a_parts:DIODE-SCHOTTKYSOD123
- FRAME1: value (none) -> FRAME-LETTERNO_PACKAGE; device A_butts:FRAME-LETTERNO_PACKAGE -> a_parts:FRAME-LETTERNO_PACKAGE
- IC1: device A_butts:ATTINY13SOIC -> a_parts:ATTINY13SOIC
- IC2: device A_butts:AMC7135SOT-89-NOTHERM -> a_parts:AMC7135SOT-89-NOTHERM
- LED, PWR: value M02JST-PTH-RA-SMALLPADS -> M02PTH-CENTERED; device A_butts:M02JST-PTH-RA-SMALLPADS -> a_parts:M02PTH-CENTERED
- R1, R2: device A_butts:RESISTORR0805 -> a_parts:RESISTORR0603-TIGHTER
