File: amc7135/amc7135-testboard-mk-1.2.brd (EAGLE design)
At the start: 24 x 20 mm, 14 parts, among them IC1 ATTiny13, IC2 AMC7135

Commit message: whoa nelly lots of boards never quite finished
Parts:
- removed IC1: ATTiny13, A_butts:SO08
- removed IC2: AMC7135, A_butts:SOT89-NOTHERM
- removed PWR: M02JST-PTH-RA-SMALLPADS, A_butts:JST-2-PH-RA-PTH-SMALLPADS
- removed R2: 1k, A_butts:RESISTOR-AXIAL-PTH-5.08MM
- removed R3: 100k, A_butts:TRIM_POT_PTH
- removed U$1: (no value), A_butts:CC-BY-SA-4.0-NO-URL
- removed U$2: (no value), A_butts:COW_SMALL
- added BRIGHT: 100k, A_butts:EVM3Y
- added BYPASS: JUMPER-PAD-2-NOYES_SILK, a_parts:PAD-JUMPER-2-NO_YES_SILK
- added JP1: M03PTH-CENTERED, a_parts:1X03-CENTERED
- added U1: Tiny13, a_parts:SO08
- added U2: AMC7135, a_parts:SOT89-NOTHERM
- AVR_ISP: value AVR_SPI_PRG_6PTH -> AVR_SPI_PRG_6SMD_TEST_POINTS; device A_butts:2X3 -> a_parts:2X3_SMD_TEST_POINTS
- C1: device A_butts:C025-024X044 -> a_parts:C0603-TIGHTER
- C2: value 10uF -> 1uF; device A_butts:C050-025X075 -> a_parts:C0603-TIGHTER
- D1: value MBRS140 -> (none); device A_butts:SMA-DIODE-SCHOTTKY -> a_parts:SOD323-SCHOTTKY
- FRAME1: value (none) -> FRAME-LETTERNO_PACKAGE; device A_butts:DUMMY -> a_parts:DUMMY
- LED: value M02JST-PTH-RA-SMALLPADS -> M02PTH-CENTERED; device A_butts:JST-2-PH-RA-PTH-SMALLPADS -> a_parts:1X02-CENTER
- R1: device A_butts:RESISTOR-AXIAL-PTH-5.08MM -> a_parts:R0603-TIGHTER
- moved D1 13.3 mm to (3.94, 7.87)
- moved R1 13.0 mm to (15.5, 8.26), turned to 0 degrees
- moved AVR_ISP 11.6 mm to (11.4, 5.08), flipped to the bottom, turned to 270 degrees
- moved C1 7.33 mm to (6.99, 7.87), turned to 90 degrees
- moved LED 2.19 mm to (21.5, 5.08), turned to 270 degrees
- moved C2 2.12 mm to (18.8, 8.26), turned to 180 degrees
Connections:
- removed net N$1: R2.P$1, R3.2
- removed net N$2: D1.A, PWR.1
- new net CTRL: JP1.1, U1.2
- new net VIN: BYPASS.1, C2.1, D1.A, JP1.3, LED.1
- net BRIGHTNESS: now also BRIGHT.S, U1.3; no longer IC1.3, R3.3
- net GND: now also BRIGHT.E, JP1.2, U1.4, U2.4@1, U2.4@2; no longer IC1.4, IC2.4@1, IC2.4@2, PWR.2, R3.1
- net LED-: now also U2.1; no longer IC2.1
- net MOSI: now also U1.5; no longer IC1.5
- net PWM: now also U1.6, U2.3; no longer IC1.6, IC2.3
- net RST: now also R1.2, U1.1; no longer IC1.1, R1.P$2
- net SCK: now also U1.7; no longer IC1.7
- net VCC: now also BRIGHT.A, BYPASS.2, R1.1, U1.8; no longer C2.1, IC1.8, LED.1, R1.P$1, R2.P$2
Routing:
- net VIN: track 0.00 -> 28.3 mm
- net VCC: track 0.00 -> 22.7 mm, vias 0 -> 1
- net RST: track 0.00 -> 14.3 mm, vias 0 -> 2
- net CTRL: track 0.00 -> 11.1 mm
- net GND: track 0.00 -> 10.6 mm, vias 0 -> 27
- net PWM: track 0.00 -> 9.89 mm, vias 0 -> 1
- net BRIGHTNESS: track 0.00 -> 8.22 mm
- net MOSI: track 0.00 -> 5.91 mm, vias 0 -> 1
- net SCK: track 0.00 -> 5.38 mm, vias 0 -> 1
- net LED-: track 0.00 -> 3.65 mm
Other:
- board size 24 x 20 mm -> 22.9 x 10.2 mm
- board text added: "!EN"
- board text added: "'7135 LED Driver"
- board text added: "GND"
- board text added: "VIN"
- board text removed: "7135 LED Driver"
- board text removed: "by schizobovine <sean@yak.net>"
