File: amc7135/amc7135-testboard-mk-1.2.sch (EAGLE design)
At the start: 12 parts, among them IC1 ATTiny13, IC2 AMC7135

Commit message: whoa nelly lots of boards never quite finished
Parts:
- removed IC1: ATTiny13, A_butts:ATTINY13SOIC
- removed IC2: AMC7135, A_butts:AMC7135SOT-89-NOTHERM
- removed PWR: M02JST-PTH-RA-SMALLPADS, A_butts:M02JST-PTH-RA-SMALLPADS
- removed R2: 1k, A_butts:RESISTORPTH-AXIAL-5.08MM
- removed R3: 100k, A_butts:TRIMPOTPTH
- added BRIGHT: 100k, A_butts:POTENTIOMETEREVM3Y
- added BYPASS: JUMPER-PAD-2-NOYES_SILK, a_parts:JUMPER-PAD-2-NOYES_SILK
- added JP1: M03PTH-CENTERED, a_parts:M03PTH-CENTERED
- added U1: Tiny13, a_parts:ATTINY13SOIC
- added U2: AMC7135, a_parts:AMC7135SOT-89-NOTHERM
- AVR_ISP: value AVR_SPI_PRG_6PTH -> AVR_SPI_PRG_6SMD_TEST_POINTS; device A_butts:AVR_SPI_PRG_6PTH -> a_parts:AVR_SPI_PRG_6SMD_TEST_POINTS
- C1: device A_butts:CAPACITOR-CERAMIC025-024X044 -> a_parts:CAPACITOR-CERAMICC0603-TIGHTER
- C2: value 10uF -> 1uF; device A_butts:CAPACITOR-CERAMIC050-025X075 -> a_parts:CAPACITOR-CERAMICC0603-TIGHTER
- D1: value MBRS140 -> (none); device A_butts:DIODE-SCHOTTKYSMA -> a_parts:DIODE-SCHOTTKYSOD323
- FRAME1: value (none) -> FRAME-LETTERNO_PACKAGE; device A_butts:FRAME-LETTERNO_PACKAGE -> a_parts:FRAME-LETTERNO_PACKAGE; DESIGNER (none) -> sean@yak.net; VERSION (none) -> v1.2
- LED: value M02JST-PTH-RA-SMALLPADS -> M02PTH-CENTERED; device A_butts:M02JST-PTH-RA-SMALLPADS -> a_parts:M02PTH-CENTERED
- R1: device A_butts:RESISTORPTH-AXIAL-5.08MM -> a_parts:RESISTORR0603-TIGHTER
Connections:
- removed net N$1: R2.1, R3.WIPER
- removed net N$2: D1.A, PWR.1
- new net CTRL: JP1.1, U1.PB3(ADC3)
- new net VIN: BYPASS.1, C2.1, D1.A, JP1.3, LED.1
- net BRIGHTNESS: now also BRIGHT.S, U1.PB4(ADC2); no longer IC1.PB4(ADC2), R3.CW
- net GND: now also BRIGHT.E, JP1.2, U1.GND, U2.GND; no longer IC1.GND, IC2.GND, PWR.2, R3.CCW
- net LED-: now also U2.LED; no longer IC2.LED
- net MOSI: now also U1.PB0(MOSI); no longer IC1.PB0(MOSI)
- net PWM: now also U1.PB1(MISO), U2.VDD; no longer IC1.PB1(MISO), IC2.VDD
- net RST: now also U1.RESET; no longer IC1.RESET
- net SCK: now also U1.PB2(SCK/ADC1); no longer IC1.PB2(SCK/ADC1)
- net VCC: now also BRIGHT.A, BYPASS.2, U1.VCC; no longer C2.1, IC1.VCC, LED.1, R2.2
Other:
- moved on the sheet: D1
