File: amc7135/amc7135-24mm-RGBW-led-driver-with-butt-mk-1.2.brd (EAGLE design)
At the start: 24 x 24 mm, 24 parts, among them U1 Tiny85-20-SMT, U10 AMC7135, U11 AMC7135, U12 AMC7135, U13 AMC7135, U2 AMC7135, U3 AMC7135, U4 AMC7135, U5 AMC7135, U6 AMC7135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

Commit message: whoops left these here?
Parts:
- removed BUTT: SPST-NO-TACT3MM-RA, a_parts:TACTILE-PTH-SIDE
- added GND, SW: M01PTH-0.8MM, a_parts:1X01-0.8MM
- moved B 45.0 mm to (28.4, 19.8)
- moved G 45.0 mm to (30.5, 19.8)
- moved R 45.0 mm to (28.4, 16.7)
- moved U7 45.0 mm to (34.6, 30.4)
- moved U8 45.0 mm to (29.8, 24.4)
- moved U9 45.0 mm to (34.6, 24.4)
- moved W 45.0 mm to (30.5, 16.7)
- moved U10 44.8 mm to (29.4, 12.3)
- moved U11 44.8 mm to (34.2, 12.3)
- moved U12 44.8 mm to (29.4, 6.30)
- moved U13 44.8 mm to (34.2, 6.30)
- moved U6 21.3 mm to (5.10, 16.5), turned to 330 degrees
- moved U2 4.18 mm to (4.00, 11.1)
- moved U3 3.14 mm to (6.50, 5.90), turned to 25 degrees
- moved U1 2.55 mm to (12.4, 4.20)
Connections:
- net BUTT: now also SW.1; no longer BUTT.1
- net GND: now also GND.1; no longer BUTT.2
Other:
- board size 24 x 24 mm -> 23 x 20 mm
