File: amc7135/amc7135-by-16-19mm-led-aux-driver-mk-1.0.1.brd (EAGLE design)
At the start: 19 x 19 mm, 20 parts, among them U1 AMC7135, U10 AMC7135, U11 AMC7135, U12 AMC7135, U13 AMC7135, U14 AMC7135, U15 AMC7135, U16 AMC7135, U2 AMC7135, U3 AMC7135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

Commit message: many WIP, left side
Parts:
- moved PWM 2.53 mm to (7.30, 7.20)
- moved GND 1.52 mm to (8.00, 12.5)
- moved LED- 1.52 mm to (11.0, 6.50)
- moved U1 0.10 mm to (9.50, 16.5)
- moved U9 0.10 mm to (9.50, 16.5)
Routing:
- net PWM: track 0.00 -> 70.7 mm, vias 0 -> 1
- net LED-: track 9.97 -> 76.3 mm, vias 0 -> 9
- net GND: track 35.5 -> 35.0 mm, vias 16 -> 14
- added copper zone on layer 1, net LED-
Other:
- board text added: "16x'7135"
- board text added: "19mm"
- board text added: "G"
- board text added: "L-"
