File: ts19370/ts19390-boost-24mm-driver-mk-1.brd (EAGLE design)
At the start: 20 x 20 mm, 14 parts, among them U1 TINY85, U2 AMC7135SOT-89, U3 AMC7135SOT-89, U4 AMC7135SOT-89, U5 AMC7135SOT-89

Commit message: faaaabulous flashlight in progress
Parts:
- removed +, 5V, B-, G-, R-, W-: M01SMD_2X3MM, A_butts:1X01_SMD_2X3MM
- removed GND: M01NOT-A-VIA-NOPE, A_butts:1X01_NOSILK_NOSTOP
- removed U1: TINY85, A_butts:QFN20
- removed U2, U3, U4, U5: AMC7135SOT-89, A_butts:SOT89
- added C2: 1uF, A_butts:C0805
- added D1, D2: B340A, A_butts:SOD123
- added D3: 10V, A_butts:SOD123
- added IC1: TS19370, A_butts:SOT26
- added L1: 22uH, A_butts:TAIYO-YUDEN-30XX
- added R2: 10-30k, A_butts:R0603
- C1: value 10uF -> 1uF
- R1: value 100k -> 4.7R
- moved C1 9.90 mm to (8.00, 13.0), turned to 90 degrees
- moved R1 1.00 mm to (15.0, 13.0), turned to 270 degrees
Connections:
- removed net 5V: +.P$1, 5V.P$1, C1.1, R1.1, U1.15
- removed net BLUE-: B-.P$1, U4.1
- removed net BLUEPWM: U1.12, U4.3
- removed net GREEN-: G-.P$1, U3.1
- removed net GREENPWM: U1.5, U3.3
- removed net RED-: R-.P$1, U2.1
- removed net REDPWM: U1.2, U2.3
- removed net WHITE-: U5.1, W-.P$1
- removed net WHITEPWM: U1.11, U5.3
- new net BATT+: D2.A
- new net LED+: C2.1, D1.C, D3.C
- new net LED-: D3.A, IC1.3, R1.2
- new net N$2: IC1.4, R2.1
- new net VCC: C1.1, D2.C, IC1.6, L1.1, R2.2
- net GND: now also C2.2, IC1.2, R1.1; no longer GND.P$1, U1.0, U1.8, U2.2, U2.4, U3.2, U3.4, U4.2, U4.4, U5.2, U5.4
- net N$1: now also D1.A, IC1.1, L1.2; no longer R1.2, U1.1
Routing:
- net 5V: track 25.5 -> 0.00 mm, vias 4 -> 0
- net BLUEPWM: track 6.13 -> 0.00 mm
- net RED-: track 4.01 -> 0.00 mm, vias 1 -> 0
- net BLUE-: track 4.01 -> 0.00 mm, vias 1 -> 0
- net WHITE-: track 4.01 -> 0.00 mm, vias 1 -> 0
- net GREEN-: track 4.01 -> 0.00 mm, vias 1 -> 0
- net N$1: track 3.92 -> 0.00 mm
- net GREENPWM: track 3.45 -> 0.00 mm
- net REDPWM: track 2.71 -> 0.00 mm
- net WHITEPWM: track 2.51 -> 0.00 mm
- removed copper zone on layer 1, net GND
- removed copper zone on layer 16, net GND
Other:
- outline, holes or cut-outs redrawn

Commit message: i'm not neve sure what i did here?
Parts:
- removed IC1: TS19370, A_butts:SOT26
- added JP1, JP2, JP3, JP4: M01PTH, A_butts:1X01
- D1, D2: device A_butts:SOD123 -> A_butts:SOD123-SCHOTTKY
- D3: device A_butts:SOD123 -> A_butts:SOD123-ZENER
Connections:
- net BATT+: now also JP1.1
- net GND: now also JP2.1; no longer IC1.2
- net LED+: now also JP3.1
- net LED-: now also JP4.1; no longer IC1.3
- net N$1: no longer IC1.1
- net N$2: no longer IC1.4
- net VCC: no longer IC1.6
Changed lines of the file:
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@@
 <setting verticaltext="up"/>
 </settings>
-<grid distance="1" unitdist="mm" unit="mm" style="lines" multiple="1" display="yes" altdistance="1" altunitdist="mm" altunit="mm"/>
+<grid distance="0.5" unitdist="mm" unit="mm" style="lines" multiple="2" display="yes" altdistance="1" altunitdist="mil" altunit="mil"/>
 <layers>
 <layer number="1" name="Top" color="4" fill="1" visible="yes" active="yes"/>
@@
 </autorouter>
 <elements>
-<element name="IC1" library="A_butts" package="SOT26" value="TS19370" x="11" y="9" smashed="yes">
-<attribute name="NAME" x="9.476" y="10.778" size="0.4064" layer="25"/>
-<attribute name="VALUE" x="11" y="9" size="0.4064" layer="27" font="vector" ratio="12" align="center"/>
-</element>
 <element name="C1" library="A_butts" package="C0805" value="1uF" x="8" y="13" rot="R90"/>
 <element name="C2" library="A_butts" package="C0805" value="1uF" x="12" y="5" rot="R270"/>
 <element name="L1" library="A_butts" package="TAIYO-YUDEN-30XX" value="22uH" x="5" y="7"/>
 <element name="R1" library="A_butts" package="R0805" value="4.7R" x="15" y="13" rot="R270"/>
-<element name="D1" library="A_butts" package="SOD123" value="B340A" x="8" y="7" rot="R90"/>
-<element name="D2" library="A_butts" package="SOD123" value="B340A" x="4" y="12" rot="R90"/>
-<element name="D3" library="A_butts" package="SOD123" value="10V" x="15" y="6" smashed="yes" rot="R90">
+<element name="D1" library="A_butts" package="SOD123-SCHOTTKY" value="B340A" x="8" y="7" rot="R90"/>
+<element name="D2" library="A_butts" package="SOD123-SCHOTTKY" value="B340A" x="4" y="12" rot="R90"/>
+<element name="D3" library="A_butts" package="SOD123-ZENER" value="10V" x="15" y="6" smashed="yes" rot="R90">
 <attribute name="NAME" x="15.889" y="6" size="0.4064" layer="25" font="vector" ratio="12" rot="R270" align="bottom-center"/>
 </element>
 <element name="R2" library="A_butts" package="R0603" value="10-30k" x="11" y="12" rot="R180"/>
+<element name="JP1" library="A_butts" package="1X01" value="M01PTH" x="-2" y="1.5"/>
+<element name="JP2" library="A_butts" package="1X01" value="M01PTH" x="-5" y="1.5"/>
+<element name="JP3" library="A_butts" package="1X01" value="M01PTH" x="-8" y="1.5"/>
+<element name="JP4" library="A_butts" package="1X01" value="M01PTH" x="-11" y="1.5"/>
 </elements>
 <signals>
 <signal name="N$1">
-<contactref element="IC1" pad="1"/>
 <contactref element="L1" pad="2"/>
 <contactref element="D1" pad="A"/>
-<wire x1="8" y1="8.9" x2="10.05" y2="7.8" width="0" layer="19" extent="1-1"/>
-<wire x1="6.1" y1="7" x2="8" y2="8.9" width="0" layer="19" extent="1-1"/>
+<wire x1="6.1" y1="7" x2="8" y2="5.1" width="0" layer="19" extent="1-1"/>
 </signal>
 <signal name="VCC">
@@
 <contactref element="D2" pad="C"/>
 <contactref element="C1" pad="1"/>
-<contactref element="IC1" pad="6"/>
 <contactref element="R2" pad="2"/>
 <wire x1="10.15" y1="12" x2="8" y2="12.05" width="0" layer="19" extent="1-1"/>
-<wire x1="10.05" y1="10.2" x2="10.15" y2="12" width="0" layer="19" extent="1-1"/>
-<wire x1="3.9" y1="7" x2="8" y2="12.05" width="0" layer="19" extent="1-1"/>
-<wire x1="4" y1="10.1" x2="3.9" y2="7" width="0" layer="19" extent="1-1"/>
+<wire x1="4" y1="13.9" x2="8" y2="12.05" width="0" layer="19" extent="1-1"/>
+<wire x1="3.9" y1="7" x2="4" y2="13.9" width="0" layer="19" extent="1-1"/>
 </signal>
 <signal name="BATT+">
 <contactref element="D2" pad="A"/>
+<contactref element="JP1" pad="1"/>
+<wire x1="-2" y1="1.5" x2="4" y2="10.1" width="0" layer="19" extent="1-1"/>
 </signal>
 <signal name="LED+">
@@
 <contactref element="C2" pad="1"/>
 <contactref element="D3" pad="C"/>
-<wire x1="15" y1="4.1" x2="12" y2="5.95" width="0" layer="19" extent="1-1"/>
-<wire x1="8" y1="5.1" x2="12" y2="5.95" width="0" layer="19" extent="1-1"/>
+<contactref element="JP3" pad="1"/>
+<wire x1="15" y1="7.9" x2="12" y2="5.95" width="0" layer="19" extent="1-1"/>
+<wire x1="8" y1="8.9" x2="12" y2="5.95" width="0" layer="19" extent="1-1"/>
+<wire x1="-8" y1="1.5" x2="8" y2="8.9" width="0" layer="19" extent="1-1"/>
 </signal>
 <signal name="LED-">
-<contactref element="IC1" pad="3"/>
 <contactref element="D3" pad="A"/>
 <contactref element="R1" pad="2"/>
-<wire x1="15" y1="7.9" x2="15" y2="12.05" width="0" layer="19" extent="1-1"/>
-<wire x1="11.95" y1="7.8" x2="15" y2="7.9" width="0" layer="19" extent="1-1"/>
+<contactref element="JP4" pad="1"/>
+<wire x1="15" y1="4.1" x2="15" y2="12.05" width="0" layer="19" extent="1-1"/>
+<wire x1="-11" y1="1.5" x2="15" y2="4.1" width="0" layer="19" extent="1-1"/>
 </signal>
 <signal name="GND">
 <contactref element="C2" pad="2"/>
-<contactref element="IC1" pad="2"/>
 <contactref element="R1" pad="1"/>
 <contactref element="C1" pad="2"/>
+<contactref element="JP2" pad="1"/>
+<wire x1="8" y1="13.95" x2="15" y2="13.95" width="0" layer="19" extent="1-1"/>
+<wire x1="12" y1="4.05" x2="15" y2="13.95" width="0" layer="19" extent="1-1"/>
+<wire x1="-5" y1="1.5" x2="12" y2="4.05" width="0" layer="19" extent="1-1"/>
 </signal>
 <signal name="N$2">
 <contactref element="R2" pad="1"/>
-<contactref element="IC1" pad="4"/>
-<wire x1="11.95" y1="10.2" x2="11.85" y2="12" width="0" layer="19" extent="1-1"/>
 </signal>
 </signals>
