File: ts19370/ts19390-boost-24mm-driver-mk-1.sch (EAGLE design)
At the start: 10 parts, among them IC1 TS19370

Commit message: faaaabulous flashlight in progress
Parts:
- removed JP1: (no value), A_butts:M08BUTTLIGHT
- D1, D2: device A_butts:DIODE-SCHOTTKYB340A -> A_butts:DIODE-SCHOTTKYSOD123
- L1: device A_butts:INDUCTORTAIYO-YUDEN-40XX -> A_butts:INDUCTORTAIYO-YUDEN-30XX
- R2: device A_butts:RESISTORR0805 -> A_butts:RESISTORR0603
Changed lines of the file:
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@@
 <layer number="19" name="Unrouted" color="6" fill="1" visible="no" active="no"/>
 <layer number="20" name="Dimension" color="15" fill="1" visible="no" active="no"/>
-<layer number="21" name="tPlace" color="15" fill="1" visible="no" active="no"/>
-<layer number="22" name="bPlace" color="14" fill="1" visible="no" active="no"/>
+<layer number="21" name="tPlace" color="7" fill="1" visible="no" active="no"/>
+<layer number="22" name="bPlace" color="7" fill="1" visible="no" active="no"/>
 <layer number="23" name="tOrigins" color="15" fill="1" visible="no" active="no"/>
 <layer number="24" name="bOrigins" color="15" fill="1" visible="no" active="no"/>
@@
 <part name="C1" library="A_butts" deviceset="CAPACITOR-CERAMIC" device="C0805" value="1uF"/>
 <part name="C2" library="A_butts" deviceset="CAPACITOR-CERAMIC" device="C0805" value="1uF"/>
-<part name="L1" library="A_butts" deviceset="INDUCTOR" device="TAIYO-YUDEN-40XX" value="22uH"/>
+<part name="L1" library="A_butts" deviceset="INDUCTOR" device="TAIYO-YUDEN-30XX" value="22uH"/>
 <part name="R1" library="A_butts" deviceset="RESISTOR" device="R0805" value="4.7R"/>
-<part name="D1" library="A_butts" deviceset="DIODE-SCHOTTKY" device="B340A" value="B340A"/>
-<part name="D2" library="A_butts" deviceset="DIODE-SCHOTTKY" device="B340A" value="B340A"/>
+<part name="D1" library="A_butts" deviceset="DIODE-SCHOTTKY" device="SOD123" value="B340A"/>
+<part name="D2" library="A_butts" deviceset="DIODE-SCHOTTKY" device="SOD123" value="B340A"/>
 <part name="D3" library="A_butts" deviceset="DIODE-ZENER" device="SOD123" value="10V"/>
-<part name="JP1" library="A_butts" deviceset="M08" device="BUTTLIGHT"/>
 <part name="GND1" library="A_butts" deviceset="GND" device=""/>
 <part name="GND2" library="A_butts" deviceset="GND" device=""/>
-<part name="R2" library="A_butts" deviceset="RESISTOR" device="R0805" value="10-30k"/>
+<part name="R2" library="A_butts" deviceset="RESISTOR" device="R0603" value="10-30k"/>
 </parts>
 <sheets>
@@
 <instance part="D2" gate="G$1" x="25.4" y="60.96"/>
 <instance part="D3" gate="G$1" x="83.82" y="45.72" rot="R90"/>
-<instance part="JP1" gate="G$1" x="111.76" y="83.82" rot="R180"/>
 <instance part="GND1" gate="1" x="58.42" y="20.32"/>
 <instance part="GND2" gate="1" x="91.44" y="43.18"/>

Commit message: i'm not neve sure what i did here?
Parts:
- removed IC1: TS19370, A_butts:TS19370
- added JP1, JP2, JP3, JP4: M01PTH, A_butts:M01PTH
Connections:
- net BATT+: now also JP1.1
- net GND: now also JP2.1; no longer IC1.GND
- net LED+: now also JP3.1
- net LED-: now also JP4.1; no longer IC1.FB
- net N$1: no longer IC1.SW
- net N$2: no longer IC1.DIM
- net VCC: no longer IC1.VIN
Changed lines of the file:
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@@
 <setting verticaltext="up"/>
 </settings>
-<grid distance="100" unitdist="mil" unit="mil" style="lines" multiple="1" display="yes" altdistance="1" altunitdist="mm" altunit="mm"/>
+<grid distance="100" unitdist="mil" unit="mil" style="lines" multiple="1" display="yes" altdistance="2" altunitdist="mil" altunit="mil"/>
 <layers>
 <layer number="1" name="Top" color="4" fill="1" visible="no" active="no"/>
@@
 </classes>
 <parts>
-<part name="IC1" library="A_butts" deviceset="TS19370" device=""/>
 <part name="C1" library="A_butts" deviceset="CAPACITOR-CERAMIC" device="C0805" value="1uF"/>
 <part name="C2" library="A_butts" deviceset="CAPACITOR-CERAMIC" device="C0805" value="1uF"/>
@@
 <part name="GND2" library="A_butts" deviceset="GND" device=""/>
 <part name="R2" library="A_butts" deviceset="RESISTOR" device="R0603" value="10-30k"/>
+<part name="JP1" library="A_butts" deviceset="M01" device="PTH"/>
+<part name="JP2" library="A_butts" deviceset="M01" device="PTH"/>
+<part name="JP3" library="A_butts" deviceset="M01" device="PTH"/>
+<part name="JP4" library="A_butts" deviceset="M01" device="PTH"/>
 </parts>
 <sheets>
@@
 </plain>
 <instances>
-<instance part="IC1" gate="G$1" x="58.42" y="43.18"/>
 <instance part="C1" gate="G$1" x="30.48" y="43.18"/>
 <instance part="C2" gate="G$1" x="91.44" y="53.34"/>
@@
 <instance part="GND2" gate="1" x="91.44" y="43.18"/>
 <instance part="R2" gate="G$1" x="40.64" y="43.18" rot="R90"/>
+<instance part="JP1" gate="G$1" x="10.16" y="60.96"/>
+<instance part="JP2" gate="G$1" x="10.16" y="25.4"/>
+<instance part="JP3" gate="G$1" x="106.68" y="60.96" rot="MR0"/>
+<instance part="JP4" gate="G$1" x="106.68" y="25.4" rot="MR0"/>
 </instances>
 <busses>
@@
 <net name="N$1" class="0">
 <segment>
-<pinref part="IC1" gate="G$1" pin="SW"/>
 <wire x1="73.66" y1="50.8" x2="73.66" y2="60.96" width="0.1524" layer="91"/>
 <pinref part="L1" gate="G$1" pin="2"/>
@@
 <wire x1="30.48" y1="48.26" x2="30.48" y2="50.8" width="0.1524" layer="91"/>
 <junction x="30.48" y="60.96"/>
-<pinref part="IC1" gate="G$1" pin="VIN"/>
 <wire x1="30.48" y1="50.8" x2="30.48" y2="60.96" width="0.1524" layer="91"/>
 <wire x1="43.18" y1="50.8" x2="40.64" y2="50.8" width="0.1524" layer="91"/>
@@
 <segment>
 <pinref part="D2" gate="G$1" pin="A"/>
-<wire x1="22.86" y1="60.96" x2="20.32" y2="60.96" width="0.1524" layer="91"/>
-<label x="20.32" y="60.96" size="1.27" layer="95" rot="R180" xref="yes"/>
+<wire x1="22.86" y1="60.96" x2="17.78" y2="60.96" width="0.1524" layer="91"/>
+<label x="22.86" y="63.5" size="1.27" layer="95" rot="R180"/>
+<pinref part="JP1" gate="G$1" pin="1"/>
 </segment>
 </net>
@@
 <wire x1="83.82" y1="48.26" x2="83.82" y2="60.96" width="0.1524" layer="91"/>
 <junction x="83.82" y="60.96"/>
-<label x="99.06" y="60.96" size="1.27" layer="95" xref="yes"/>
+<label x="99.06" y="63.5" size="1.27" layer="95" rot="R180"/>
 <wire x1="91.44" y1="60.96" x2="99.06" y2="60.96" width="0.1524" layer="91"/>
+<pinref part="JP3" gate="G$1" pin="1"/>
 </segment>
 </net>
 <net name="LED-" class="0">
 <segment>
-<pinref part="IC1" gate="G$1" pin="FB"/>
 <pinref part="D3" gate="G$1" pin="A"/>
 <wire x1="73.66" y1="35.56" x2="83.82" y2="35.56" width="0.1524" layer="91"/>
 <wire x1="83.82" y1="35.56" x2="83.82" y2="43.18" width="0.1524" layer="91"/>
 <pinref part="R1" gate="G$1" pin="2"/>
-<wire x1="93.98" y1="25.4" x2="83.82" y2="25.4" width="0.1524" layer="91"/>
+<wire x1="99.06" y1="25.4" x2="83.82" y2="25.4" width="0.1524" layer="91"/>
 <wire x1="83.82" y1="25.4" x2="76.2" y2="25.4" width="0.1524" layer="91"/>
 <wire x1="83.82" y1="35.56" x2="83.82" y2="25.4" width="0.1524" layer="91"/>
 <junction x="83.82" y="35.56"/>
 <junction x="83.82" y="25.4"/>
-<label x="93.98" y="25.4" size="1.27" layer="95" xref="yes"/>
+<label x="93.98" y="22.86" size="1.27" layer="95"/>
+<pinref part="JP4" gate="G$1" pin="1"/>
 </segment>
 </net>
@@
 </segment>
 <segment>
-<pinref part="IC1" gate="G$1" pin="GND"/>
 <wire x1="30.48" y1="25.4" x2="58.42" y2="25.4" width="0.1524" layer="91"/>
 <wire x1="58.42" y1="25.4" x2="58.42" y2="27.94" width="0.1524" layer="91"/>
@@
 <wire x1="30.48" y1="38.1" x2="30.48" y2="25.4" width="0.1524" layer="91"/>
 <junction x="30.48" y="25.4"/>
-<wire x1="30.48" y1="25.4" x2="20.32" y2="25.4" width="0.1524" layer="91"/>
-<label x="20.32" y="25.4" size="1.27" layer="95" rot="R180" xref="yes"/>
+<wire x1="30.48" y1="25.4" x2="17.78" y2="25.4" width="0.1524" layer="91"/>
+<label x="20.32" y="22.86" size="1.27" layer="95"/>
+<pinref part="JP2" gate="G$1" pin="1"/>
 </segment>
 </net>
@@
 <pinref part="R2" gate="G$1" pin="1"/>
 <wire x1="40.64" y1="38.1" x2="40.64" y2="35.56" width="0.1524" layer="91"/>
-<pinref part="IC1" gate="G$1" pin="DIM"/>
 <wire x1="40.64" y1="35.56" x2="43.18" y2="35.56" width="0.1524" layer="91"/>
 </segment>
