File: mp3412/mp3412-boost-driver-13mm-mk-1.0.brd (EAGLE design)
At the start: 13 x 13 mm, 10 parts, among them U2 MP3412

Commit message: board tweak, flashlight test program in arduino
Routing:
- added copper zone on layer 16, net GND
Changed lines of the file:
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@@
+<vertex x="13" y="0"/>
+</polygon>
+<polygon width="0.1524" layer="16" isolate="0.3048" rank="6">
+<vertex x="0" y="0"/>
+<vertex x="0" y="13"/>
+<vertex x="13" y="13"/>
 <vertex x="13" y="0"/>
 </polygon>
