File: rgb-direct/rgbw-direct-driver-mk-1.0.brd (EAGLE design)
At the start: 17 x 17 mm, 16 parts, among them Q1 IRLM2502, Q2 IRLM2502, Q3 IRLM2502, Q4 IRLM2502, U1 Tiny13

Commit message: wip
Parts:
- Q1, Q2, Q3, Q4: device a_parts:SOT23 -> a_parts:SOT23-CLOSER
- moved R1 12.0 mm to (14.5, 8.50), turned to 270 degrees
- moved C2 6.80 mm to (6.50, 14.5), turned to 180 degrees
- moved Q4 6.46 mm to (3.70, 6.80), turned to 90 degrees
- moved D1 3.81 mm to (5.00, 10.5), turned to 180 degrees
- moved C1 3.76 mm to (5.50, 12.5)
- moved W 3.35 mm to (2.00, 8.50), turned to 180 degrees
- moved U1 3.04 mm to (10.0, 8.50)
- moved G 2.00 mm to (8.50, 3.00), turned to 90 degrees
- moved B 1.98 mm to (13.5, 5.00)
- moved Q2 1.80 mm to (6.00, 3.50), turned to 180 degrees
- moved Q3 1.65 mm to (11.1, 3.40)
- moved + 1.30 mm to (6.50, 8.70)
- moved R 1.08 mm to (9.00, 14.5)
- moved Q1 1.02 mm to (11.0, 13.7)
Connections:
- net PWM_B: now also R1.D2; no longer R1.B2
- net PWM_G: now also R1.C2; no longer R1.A2
- net PWM_R: now also R1.A2; no longer R1.C2
- net PWM_W: now also R1.B2; no longer R1.D2
Routing:
- net GREEN: track 0.00 -> 2.71 mm
- net BLUE: track 0.00 -> 2.18 mm
- net WHITE: track 0.00 -> 1.99 mm
