File: rgb-direct/rgbw-direct-driver-mk-1.0.sch (EAGLE design)
At the start: 16 parts, among them Q1 IRLM2502, Q2 IRLM2502, Q3 IRLM2502, Q4 IRLM2502, U1 Tiny13

Commit message: wip
Parts:
- Q1, Q2, Q3, Q4: device a_parts:MOSFET-NCHANNELIRLML2502 -> a_parts:MOSFET-NCHANNELIRLML2502-SMOL
Connections:
- net PWM_B: now also R1D.2; no longer R1B.2
- net PWM_G: now also R1C.2; no longer R1A.2
- net PWM_R: now also R1A.2; no longer R1C.2
- net PWM_W: now also R1B.2; no longer R1D.2
Other:
- moved on the sheet: R1A, R1B, R1C, R1D
Changed lines of the file:
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@@
 <part name="G" library="a_parts" deviceset="M01" device="SMD-1.25MM-DIA" value="M01SMD-1.25MM-DIA"/>
 <part name="B" library="a_parts" deviceset="M01" device="SMD-1.25MM-DIA" value="M01SMD-1.25MM-DIA"/>
-<part name="Q1" library="a_parts" deviceset="MOSFET-NCHANNEL" device="IRLML2502" value="IRLM2502"/>
-<part name="Q2" library="a_parts" deviceset="MOSFET-NCHANNEL" device="IRLML2502" value="IRLM2502"/>
-<part name="Q3" library="a_parts" deviceset="MOSFET-NCHANNEL" device="IRLML2502" value="IRLM2502"/>
-<part name="Q4" library="a_parts" deviceset="MOSFET-NCHANNEL" device="IRLML2502" value="IRLM2502"/>
+<part name="Q1" library="a_parts" deviceset="MOSFET-NCHANNEL" device="IRLML2502-SMOL" value="IRLM2502"/>
+<part name="Q2" library="a_parts" deviceset="MOSFET-NCHANNEL" device="IRLML2502-SMOL" value="IRLM2502"/>
+<part name="Q3" library="a_parts" deviceset="MOSFET-NCHANNEL" device="IRLML2502-SMOL" value="IRLM2502"/>
+<part name="Q4" library="a_parts" deviceset="MOSFET-NCHANNEL" device="IRLML2502-SMOL" value="IRLM2502"/>
 <part name="R1" library="a_parts" deviceset="RESISTOR-ARRAY-4" device="YC164" value="10K"/>
 </parts>
@@
 <instance part="Q3" gate="G$1" x="121.92" y="68.58"/>
 <instance part="Q4" gate="G$1" x="165.1" y="68.58"/>
-<instance part="R1" gate="A" x="71.12" y="60.96" rot="R90"/>
-<instance part="R1" gate="B" x="111.76" y="60.96" rot="R90"/>
-<instance part="R1" gate="C" x="30.48" y="60.96" rot="R90"/>
-<instance part="R1" gate="D" x="154.94" y="60.96" rot="R90"/>
+<instance part="R1" gate="A" x="30.48" y="60.96" rot="R90"/>
+<instance part="R1" gate="B" x="154.94" y="60.96" rot="R90"/>
+<instance part="R1" gate="C" x="71.12" y="60.96" rot="R90"/>
+<instance part="R1" gate="D" x="111.76" y="60.96" rot="R90"/>
 </instances>
 <busses>
@@
 <wire x1="30.48" y1="53.34" x2="40.64" y2="53.34" width="0.1524" layer="91"/>
 <pinref part="R1" gate="D" pin="1"/>
-<wire x1="154.94" y1="55.88" x2="154.94" y2="53.34" width="0.1524" layer="91"/>
+<wire x1="111.76" y1="53.34" x2="111.76" y2="55.88" width="0.1524" layer="91"/>
+<junction x="111.76" y="53.34"/>
+<pinref part="R1" gate="B" pin="1"/>
+<wire x1="154.94" y1="53.34" x2="154.94" y2="55.88" width="0.1524" layer="91"/>
 <junction x="154.94" y="53.34"/>
 <pinref part="R1" gate="C" pin="1"/>
-<wire x1="30.48" y1="55.88" x2="30.48" y2="53.34" width="0.1524" layer="91"/>
-<pinref part="R1" gate="A" pin="1"/>
 <wire x1="71.12" y1="55.88" x2="71.12" y2="53.34" width="0.1524" layer="91"/>
 <junction x="71.12" y="53.34"/>
-<pinref part="R1" gate="B" pin="1"/>
-<wire x1="111.76" y1="55.88" x2="111.76" y2="53.34" width="0.1524" layer="91"/>
-<junction x="111.76" y="53.34"/>
+<pinref part="R1" gate="A" pin="1"/>
+<wire x1="30.48" y1="53.34" x2="30.48" y2="55.88" width="0.1524" layer="91"/>
 </segment>
 </net>
@@
 <pinref part="Q1" gate="G$1" pin="G"/>
 <wire x1="27.94" y1="68.58" x2="30.48" y2="68.58" width="0.1524" layer="91"/>
-<pinref part="R1" gate="C" pin="2"/>
+<pinref part="R1" gate="A" pin="2"/>
 <wire x1="30.48" y1="68.58" x2="33.02" y2="68.58" width="0.1524" layer="91"/>
 <wire x1="30.48" y1="68.58" x2="30.48" y2="66.04" width="0.1524" layer="91"/>
@@
 <pinref part="Q4" gate="G$1" pin="G"/>
 <wire x1="152.4" y1="68.58" x2="154.94" y2="68.58" width="0.1524" layer="91"/>
-<pinref part="R1" gate="D" pin="2"/>
+<pinref part="R1" gate="B" pin="2"/>
 <wire x1="154.94" y1="68.58" x2="157.48" y2="68.58" width="0.1524" layer="91"/>
-<wire x1="154.94" y1="68.58" x2="154.94" y2="66.04" width="0.1524" layer="91"/>
+<wire x1="154.94" y1="66.04" x2="154.94" y2="68.58" width="0.1524" layer="91"/>
 <junction x="154.94" y="68.58"/>
 </segment>
@@
 <pinref part="Q2" gate="G$1" pin="G"/>
 <wire x1="68.58" y1="68.58" x2="71.12" y2="68.58" width="0.1524" layer="91"/>
-<pinref part="R1" gate="A" pin="2"/>
+<pinref part="R1" gate="C" pin="2"/>
 <wire x1="71.12" y1="68.58" x2="73.66" y2="68.58" width="0.1524" layer="91"/>
 <wire x1="71.12" y1="68.58" x2="71.12" y2="66.04" width="0.1524" layer="91"/>
@@
 <pinref part="Q3" gate="G$1" pin="G"/>
 <wire x1="109.22" y1="68.58" x2="111.76" y2="68.58" width="0.1524" layer="91"/>
-<pinref part="R1" gate="B" pin="2"/>
+<pinref part="R1" gate="D" pin="2"/>
 <wire x1="111.76" y1="68.58" x2="114.3" y2="68.58" width="0.1524" layer="91"/>
 <wire x1="111.76" y1="68.58" x2="111.76" y2="66.04" width="0.1524" layer="91"/>
