File: rw-directish/2LD-20-mk-1.1.1.brd (EAGLE design)
At the start: 20 x 20 mm, 28 parts, among them U1 Tiny25, U10 AMC7135, U11 AMC7135, U12 AMC7135, U13 AMC7135, U14 AMC7135, U15 AMC7135, U16 V_REG_SOT-23-5AP2112, U2 AMC7135, U3 AMC7135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

Commit message: fix cream layer for stencils
Parts:
- U16: value V_REG_SOT-23-5AP2112 -> (none)
Changed lines of the file:
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@@
 <layer number="46" name="Milling" color="3" fill="1" visible="yes" active="yes"/>
 <layer number="47" name="Measures" color="5" fill="1" visible="yes" active="yes"/>
-<layer number="48" name="Document" color="7" fill="1" visible="yes" active="yes"/>
-<layer number="49" name="Reference" color="7" fill="1" visible="yes" active="yes"/>
+<layer number="48" name="Document" color="6" fill="1" visible="yes" active="yes"/>
+<layer number="49" name="Reference" color="6" fill="1" visible="yes" active="yes"/>
 <layer number="50" name="dxf" color="7" fill="1" visible="no" active="no"/>
-<layer number="51" name="tDocu" color="7" fill="1" visible="yes" active="yes"/>
-<layer number="52" name="bDocu" color="7" fill="1" visible="yes" active="yes"/>
+<layer number="51" name="tDocu" color="6" fill="1" visible="yes" active="yes"/>
+<layer number="52" name="bDocu" color="5" fill="1" visible="yes" active="yes"/>
 <layer number="53" name="tGND_GNDA" color="7" fill="9" visible="no" active="no"/>
 <layer number="54" name="bGND_GNDA" color="1" fill="9" visible="no" active="no"/>
@@
 <layer number="98" name="Guide" color="6" fill="1" visible="no" active="no"/>
 <layer number="99" name="SpiceOrder" color="7" fill="1" visible="no" active="no"/>
-<layer number="100" name="Muster" color="7" fill="1" visible="no" active="yes"/>
+<layer number="100" name="Muster" color="7" fill="1" visible="yes" active="yes"/>
 <layer number="101" name="Patch_Top" color="12" fill="4" visible="yes" active="yes"/>
 <layer number="102" name="Vscore" color="7" fill="1" visible="yes" active="yes"/>
@@
 </element>
 <element name="U15" library="a_parts" package="SOT89-NOTHERM-ROUNDED-LESS" value="AMC7135" x="2.9" y="10" smashed="yes" rot="R90"/>
-<element name="U16" library="a_parts" package="SOT23-5" value="V_REG_SOT-23-5AP2112" x="11" y="8.4" smashed="yes"/>
+<element name="U16" library="a_parts" package="SOT23-5" value="" x="11" y="8.4" smashed="yes"/>
 <element name="C2" library="a_parts" package="C0402" value="1u" x="8.5" y="8" smashed="yes" rot="R90">
 <attribute name="NAME" x="8.50000625" y="9.250003125" size="0.8" layer="25" font="vector" ratio="10" align="bottom-center"/>
