File: lt3477/lt3477-buck-boost-flashlight-driver-17mm-mk-1.0.sch (EAGLE design)
At the start: 24 parts, among them U1 Tiny25, U2 LT3477

Commit message: bunch of new board word
Parts:
- removed C2: 10uF, a_parts:CAPACITOR-CERAMICC0603-TIGHTER
- removed C5: 33nF, a_parts:CAPACITOR-CERAMICC0402
- removed R4: R068, a_parts:RESISTORR0805-TIGHTER
- removed R7: 22K, a_parts:RESISTORR0402
- removed R8: 1K, a_parts:RESISTORR0402
- added C55: 1uF, a_parts:CAPACITOR-CERAMICC0603-TIGHTER
- added C66: 1uF, a_parts:CAPACITOR-CERAMICC0402
- added Q1, Q2: 2N7002, a_parts:MOSFET-NCHANNELIRLML2502
- added R30: 4.7K, a_parts:RESISTORR0603-TIGHTER
- C4: value 1uF -> 33nF
- C6: value 4.7nF -> 10nF
- L1: value 10uH -> 4.7uH
- R1: value 10K -> R068; device a_parts:RESISTORR0402 -> a_parts:RESISTORR0805-TIGHTER
- R3: value 4.7K -> 22K; device a_parts:RESISTORR0603-TIGHTER -> a_parts:RESISTORR0402
- U1: device a_parts:ATTINY45TINY25-SOICN-NARROWER -> a_parts:ATTINY1310M1
- renumbered R2 to R20
Connections:
- removed net N$6: C6.1, R8.1
- removed net N$7: R8.2, U2.VC
- net GND: now also C55.2, C66.2, R30.1; no longer C2.2, C5.2, L-.1, R7.1
- net ISP2: now also R1.2; no longer R4.2
- net LED+: now also R1.1; no longer R4.1
- net N$1: now also R3.2; no longer R7.2
- net N$2: now also C6.1, U2.VC; no longer R1.1, U1.RESET
- net N$3: now also R30.2; no longer R3.2
- net N$4: now also C4.1; no longer C5.1
- net N$5: now also C66.1; no longer C4.1
- net PWM: now also U2.!SHDN
- net VBAT: now also C1.1, L-.1; no longer C2.1
- net VCC: now also C55.1; no longer C1.1, R1.2
Other:
- moved on the sheet: C1, C3, C4, D2, L+, L-, L1, R1, R3, R5, R6, U1
