File: ltc3783/ltc3783-boost-driver-test-mk-1.0.0.sch (EAGLE design)
At the start: 8 parts, among them U1 Tiny25

Commit message: bunch of new board word
Parts:
- removed +, -: M01NOT-A-VIA-NOPE, a_parts:M01NOT-A-VIA-NOPE
- added C2: (no value), a_parts:CAPACITOR-CERAMICC0805-TIGHTER
- added C3: 4.7uF, a_parts:CAPACITOR-CERAMICC0603-TIGHTER
- added C4: 0.1uF, a_parts:CAPACITOR-CERAMICC0603-TIGHTER
- added C_TINY: 1uF, a_parts:CAPACITOR-CERAMICC0402
- added D2: (no value), a_parts:DIODE-SCHOTTKYSOD323
- added LED+, LED-: M01NOT-A-VIA-NOPE, a_parts:M01NOT-A-VIA-NOPE
- added Q1: PSMN4R0-30YLD, a_parts:MOSFET-NCHANNELLFPAK33
- added R2: 21.5K, a_parts:RESISTORR0603-TIGHTER
- added R3: 66.5K, a_parts:RESISTORR0603-TIGHTER
- added R4: 17.4K, a_parts:RESISTORR0603-TIGHTER
- added R5: 698K, a_parts:RESISTORR0603-TIGHTER
- added R6: 11.5K, a_parts:RESISTORR0603-TIGHTER
- added R7: R010, a_parts:RESISTORR0805-TIGHTER
- added R8: R050, a_parts:RESISTORR0805-TIGHTER
- added U2: LTC3783DHD, a_parts:LTC3783DHD
- C1: value 1uF -> 3.3uF; device a_parts:CAPACITOR-CERAMICC0402 -> a_parts:CAPACITOR-CERAMICC0805-TIGHTER
- L1: value (none) -> 10uH; device a_parts:INDUCTORXFL4020 -> a_parts:INDUCTORXAL40X0
- R1: value 10K -> 1M; device a_parts:RESISTORR0402 -> a_parts:RESISTORR0603-TIGHTER
- U1: device a_parts:ATTINY45TINY85-20-QFN -> a_parts:ATTINY45TINY25-SOICN-NARROWER
Connections:
- new net GATE: Q1.G, U2.GATE
- new net ILIM: R3.2, R4.2, U2.ILIM
- new net INTVCC: C3.1, U2.INTVCC
- new net ITH: C4.1, U2.ITH
- new net LED-/FBP: LED-.1, R8.1, U2.FBP
- new net N$2: C2.1, D2.C, LED+.1, R5.1
- new net N$4: R2.2, U2.FREQ
- new net OV/FB: R5.2, R6.2, U2.OV/FB
- new net PWM: U1.PB1(MISO)
- new net RUN: R1.1, U2.RUN
- new net SENSE: Q1.S, R7.2, U2.SENSE
- new net VREF: R4.1, U2.VREF
- net GND: now also C2.2, C3.2, C4.2, C_TINY.2, R2.1, R3.1, R6.1, R7.1, U2.GND; no longer -.1
- net N$1: now also D2.A, L1.2, Q1.D; no longer R1.2, U1.RESET
- net VBAT: now also C1.1, L1.1, R1.2, R8.2, U2.FBN, U2.VIN; no longer +.1
- net VCC: now also C_TINY.1; no longer C1.1, R1.1
Other:
- moved on the sheet: C1, D1, L1, R1, U1
