File: tps63020/tps63020-buck-boost-flashlight-driver-17mm-mk-1.0.0.brd (EAGLE design)
At the start: 17 x 17 mm, 24 parts, among them Q1 2N7002, Q2 2N7002, U1 Tiny25, U2 LT3477

Commit message: bunch of new board word
Parts:
- removed +, L+, L-: M01PTH-1MM-CIR-NS, a_parts:1X01-1MM-CIR-NS
- removed -: M01NOT-A-VIA-NOPE, a_parts:1X01_NOSILK_NOSTOP
- removed C6: 10nF, a_parts:C0402
- removed Q1, Q2: 2N7002, a_parts:SOT23
- removed R5: 200K, a_parts:R0402
- removed R6: 10K, a_parts:R0402
- added C2: 10uF, a_parts:C0603-TIGHTER
- added C5: 1nF, a_parts:C0402
- added LED+, LED-: M01PTH-1MM-CIR-NS, a_parts:1X01-1MM-CIR-NS
- added R2: 13mOhm, a_parts:R0805-TIGHTER
- added U$1: INA190RSW, a_parts:UQFN-10
- added U3: INA193, a_parts:SOT23-5
- C1: value 10uF -> 100nF; device a_parts:C0603-TIGHTER -> a_parts:C0402
- C3: value 2.2uF -> 1uF; device a_parts:C0603-TIGHTER -> a_parts:C0402
- C4: value 33nF -> 22uF; device a_parts:C0402 -> a_parts:C0603-TIGHTER
- D2: value BAT60A -> BAT54C; device a_parts:SOD323-SCHOTTKY -> a_parts:SOT23
- L1: value 4.7uH -> 2.2uH; device a_parts:XAL40X0 -> a_parts:XAL50X0
- R1: value R068 -> 384R; device a_parts:R0805-TIGHTER -> a_parts:R0402
- R3: value 22K -> 6.34K
- U1: value Tiny25 -> TPS63020DSJ; device a_parts:QFN10(2X5) -> a_parts:VSON-14-4MMX3MM
- U2: value LT3477 -> ATTINY1310M1; device a_parts:QFN20-LTC -> a_parts:QFN10(2X5)
- moved R3 67.8 mm to (-43.0, -17.5)
- moved C3 65.6 mm to (-35.0, -17.5)
- moved C4 65.1 mm to (-39.0, -17.0)
- moved C1 54.8 mm to (-23.5, -14.0)
- moved D2 49.2 mm to (-15.0, -13.0)
- moved L1 43.9 mm to (-10.0, -1.00)
- moved R1 43.3 mm to (-31.5, -14.0), turned to 0 degrees
- moved U2 15.6 mm to (-3.50, 1.50), turned to 0 degrees
- moved U1 14.8 mm to (-4.50, -3.00), turned to 0 degrees
Connections:
- removed net FBN: R5.1, R6.2, U2.8
- removed net ISP2: C3.1, D2.C, R1.2, R5.2, U2.13
- removed net N$1: R3.2, U2.4
- removed net N$2: C6.1, U2.7
- removed net N$4: C4.1, U2.6
- removed net N$9: U2.10, U2.9
- removed net SW: D2.A, L1.P$2, U2.18, U2.19
- new net FB: R3.2, U3.1
- new net FB_LOWPASS: C5.1, R3.1, U1.3
- new net L1: L1.P$1, U1.8, U1.9
- new net L2: L1.P$2, U1.6, U1.7
- new net SHUNT_VP: C3.1, D2.3, R1.2, U3.5
- new net VINA: C1.1, U1.1, U1.12
- new net VOUT: C4.1, D2.1, R2.1, U1.4, U1.5, U3.3
- net GND: now also C2.2, C5.2, LED-.1, R1.1, U1.2, U1.PAD1, U1.PAD2, U1.PAD3, U1.PAD4, U1.PAD5, U1.PAD6, U1.PAD7, U1.PAD8, U1.PADCENTER, U2.5, U3.2; no longer -.P$1, C6.2, R3.1, R6.1, U1.5, U1.PAD, U2.17
- net LED+: now also LED+.1, R2.2, U3.4; no longer L+.1, R1.1, U2.14
- net N$3: now also U2.9; no longer U1.9
- net N$5: now also U2.2; no longer U1.2
- net PWM: now also U1.13, U2.7; no longer U1.7, U2.5
- net VBAT: now also C2.1, D2.2, U1.10, U1.11; no longer +.1, C1.1, L-.1, L1.P$1, U2.15, U2.16, U2.3
- net VCC: now also U2.10; no longer U1.10
Other:
- board text added: "TPS63020 Buck-Boost Flashlight Driver"
- board text removed: "LT3477 Buck-Boost Flashlight Driver"
