File: tps63020/tps63020-buck-boost-flashlight-driver-17mm-mk-1.0.1.sch (EAGLE design)
At the start: 16 parts, among them Q1 PSMN2R4-30MLD, U1 ATTINY13a, U2 PAM2803

Commit message: bunch of new board word
Parts:
- removed A, K: M01PTH-1MM-CIR-NS, a_parts:M01PTH-1MM-CIR-NS
- removed Q1: PSMN2R4-30MLD, a_parts:MOSFET-NCHANNELLFPAK33
- added C3, C6, C7, C8: 1uF, a_parts:CAPACITOR-CERAMICC0402
- added C4: 1nF, a_parts:CAPACITOR-CERAMICC0402
- added C5: 22uF, a_parts:CAPACITOR-CERAMICC0805-TIGHTER
- added J1: AVR_SPI_PRG_6SMD-1.27MM, a_parts:AVR_SPI_PRG_6SMD-1.27MM
- added U3: INA190A1RSW, a_parts:INA190RSW
- added U4: V_REG_ENTLV700, a_parts:V_REG_ENTLV700
- +, -: value M01NOT-A-VIA-NOPE -> M01PTH-1MM-CIR-NS; device a_parts:M01NOT-A-VIA-NOPE -> a_parts:M01PTH-1MM-CIR-NS
- C1: value 10uF -> 100nF; device a_parts:CAPACITOR-CERAMICC0805-TIGHTER -> a_parts:CAPACITOR-CERAMICC0402
- C2: value 22uF -> 10uF
- D1: value BAT60 -> BAT165
- FRAME1: VERSION v1.1 -> v1.2
- L1: value 2.2uF -> 1uH; device a_parts:INDUCTORXFL4020 -> a_parts:INDUCTORXAL50X0
- R1: value 0R1 -> 13mOhm; device a_parts:RESISTORR0603-TIGHTER -> a_parts:RESISTORR0805-TIGHTER
- R2: value 150K -> 19.1K; device a_parts:RESISTORR0603-TIGHTER -> a_parts:RESISTORR0402
- R3: value 33K -> 4.7K; device a_parts:RESISTORR0603-TIGHTER -> a_parts:RESISTORR0402
- R4: value 33R -> 6.34K; device a_parts:RESISTORR0603-TIGHTER -> a_parts:RESISTORR0402
- U1: value ATTINY13a -> TPS63020DSJ; device a_parts:ATTINY13SOIC-NARROWER -> a_parts:TPS63020DSJ
- U2: value PAM2803 -> ATTINY25-20MU; device a_parts:PAM2803SOT23-6 -> a_parts:ATTINY45TINY85-20-QFN
Connections:
- removed net !SHDN: U1.PB3(ADC3), U2.!SHDN
- removed net GATE: Q1.G, R3.2, R4.2
- removed net LED-: K.1, Q1.D
- removed net PWM: R4.1, U1.PB1(MISO)
- removed net SW: D1.A, L1.1, U2.SW
- new net ALTPWM/MOSI: J1.MOSI, U2.PB0(MOSI)
- new net FB_LOWPASS: C4.2, R4.1, U1.FB
- new net L1: L1.1, U1.L1
- new net L2: L1.2, U1.L2
- new net N$5: C7.1, U2.PB3(ADC3)
- new net PWM/MISO: J1.MISO, U1.PS/SYNC, U2.PB1(MISO)
- new net RST: J1.RST, U2.RESET
- new net VBAT_RECT: D1.C, R2.1, U4.EN, U4.IN
- new net VCC: C3.1, C6.2, C8.1, J1.VCC, U2.VCC, U3.EN, U3.VCC, U4.OUT
- new net VDIV/SCK: J1.SCK, R2.2, R3.2, U2.PB2(SCK/ADC1)
- new net VINA: C1.1, U1.EN, U1.VINA
- new net VOUT: C5.1, R1.1, U1.VOUT, U3.VIN+
- net FB: now also R4.2, U3.OUT; no longer Q1.S, R1.2, R3.1, U2.FB
- net GND: now also C3.2, C4.1, C5.2, C6.1, C7.2, C8.2, J1.GND, R3.1, U1.PGND, U3.GND, U3.REF, U4.GND; no longer R1.1, R2.1
- net LED+: now also +.1, R1.2, U3.VIN-; no longer A.1, C2.1, D1.C, U2.VO
- net VBAT: now also C2.1, D1.A, U1.VIN; no longer +.1, C1.1, L1.2, R2.2, U1.VCC, U2.VIN
Other:
- note added: "0.5V R1 = ---------- Gain * Iout"
- note added: "1 f = ----------- 2*pi*R4*C4"
- note added: "Gain = 25 (INA190A1) Iout = 1.5A R1 = 13 mOhm"
- note added: "low-pass filter"
- note added: "off-time capacitor"
- note removed: "0.095V Iout = ------ R1"
- note removed: "0R27 = 352 mA 0R22 = 432 mA 0R20 = 475 mA 0R18 = 528 mA 0R15 = 633 mA 0R12 = 792 mA 0R10 = 950 mA"
- moved on the sheet: +, -, C1, C2, D1, L1, R1, R2, R3, R4
