File: mp28164/mp28164-buck-boost-flashlight-driver-17mm-mk-1.0.0.brd (EAGLE design)
At the start: 17.6 x 17.6 mm, 20 parts, among them J1 AVR_SPI_PRG_6SMD-1.27MM, U1 MPS28164, U2 ATTINY25-20MU, U4 V_REG_ENTLV700

Commit message: whole bunch of crap in here
Parts:
- removed C2: 10uF, a_parts:C0805-TIGHTER
- removed C4: 1uF, a_parts:C0402
- added C6: 1uF, a_parts:C0402
- added C8: 6.8nF, a_parts:C0402
- added R10: 68k, a_parts:R0402
- added R5: 75k, a_parts:R0402
- added R6: 4.7k, a_parts:R0402
- added R7, R8: 1k, a_parts:R0402
- added R9: 750K, a_parts:R0402
- +, -: value M01PTH-1MM-CIR-NS -> M01SMD-1.6MMX3.2MM-NS; device a_parts:1X01-1MM-CIR-NS -> a_parts:1X01-SMD-1.6MMX3.2MM-NS
- C1: value 100nF -> 47uF; device a_parts:C0402 -> a_parts:C1206
- C3: value 22uF -> 47uF; device a_parts:C0805-TIGHTER -> a_parts:C1206
- C5: value 1uF -> 100nF
- L1: device a_parts:XAR7030 -> a_parts:XAL7070
- R1: value 13mOhm -> 10mOhm
- R4: value 19.1K -> 360k
- U3: value (none) -> OPA333
- moved R4 19.5 mm to (6.00, 14.0), flipped to the bottom, turned to 270 degrees
- moved U4 18.2 mm to (4.50, 5.50), flipped to the bottom, turned to 270 degrees
- moved C7 17.4 mm to (4.50, 7.50), flipped to the bottom, turned to 180 degrees
- moved J1 15.6 mm to (9.00, 14.0)
- moved C5 13.7 mm to (8.30, 2.50), turned to 270 degrees
- moved C1 13.5 mm to (6.00, 5.50), flipped to the top, turned to 270 degrees
- moved D1 13.1 mm to (7.00, 5.00), flipped to the bottom, turned to 270 degrees
- moved U2 11.8 mm to (14.0, 9.00), flipped to the bottom, turned to 90 degrees
- moved U3 10.8 mm to (4.00, 9.50), flipped to the bottom, turned to 90 degrees
- moved R1 10.7 mm to (4.00, 12.0), turned to 270 degrees
- moved R3 7.50 mm to (14.0, 5.00)
- moved R2 6.32 mm to (12.0, 5.00), turned to 180 degrees
- moved - 3.81 mm to (2.50, 9.00), turned to 180 degrees
- moved + 3.42 mm to (15.5, 9.00), turned to 180 degrees
- moved C3 1.50 mm to (12.0, 5.50)
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Connections:
- removed net N$1: U3.3
- removed net N$5: C7.1, U2.2
- new net FB: R10.1, R7.1, R9.2, U1.6
- new net LOWPASS: C8.2, R4.1, R8.2
- new net OPAMP-: R4.2, R5.1, R6.2, U3.3
- new net OPAMP_OUT: R5.2, R7.2, U3.4
- net ALTPWM/MOSI: now also R8.1
- net GND: now also C5.2, C6.2, C8.1, R10.2, R6.1; no longer C2.2, C4.2
- net LED-: now also -.P$1; no longer -.1
- net VBAT: now also C1.1; no longer C2.1
- net VCC: now also C6.1, C7.1; no longer C4.1
- net VDD: now also C5.1; no longer C1.1
- net VOUT: now also +.P$1, R9.1; no longer +.1
Routing:
- net VCC: track 0.00 -> 27.6 mm, vias 0 -> 3
- net VDIV/SCK: track 0.00 -> 17.8 mm, vias 0 -> 2
- net PWM/MISO: track 0.00 -> 16.5 mm, vias 0 -> 3
- net ALTPWM/MOSI: track 0.00 -> 11.5 mm, vias 0 -> 2
- net RST: track 0.00 -> 11.2 mm
- net OPAMP_OUT: track 0.00 -> 10.9 mm, vias 0 -> 2
- net VBAT_RECT: track 0.00 -> 10.2 mm
- net LOWPASS: track 0.00 -> 9.83 mm
- net FB: track 0.00 -> 8.94 mm, vias 0 -> 1
- net OPAMP-: track 0.00 -> 5.75 mm
- net VDD: track 0.00 -> 1.99 mm
- net VBAT: track 0.00 -> 1.72 mm, vias 0 -> 7
- net LED-: track 0.00 -> 1.46 mm, vias 0 -> 1
- net VOUT: track 0.00 -> 1.00 mm
- added copper zone on layer 15, net GND
- added copper zone on layer 1, net L1
- added copper zone on layer 1, net L2
- added copper zone on layer 1, net LED-
- added copper zone on layer 1, net VBAT
- added copper zone on layer 1, net VOUT
Other:
- board text added: "LED Driver"
- board text added: "MP28614"
- board text removed: "TPS63020 Buck-Boost LED Driver"
