File: mp28164/mp28164-buck-boost-flashlight-driver-tester-mk-1.0.1.opamp.only.brd (EAGLE design)
At the start: 20 x 20 mm, 13 parts, among them U3 OPA333

Commit message: whole bunch of crap in here
Parts:
- added LED1: LED3MM, a_parts:LED3MM
- added U1: (no value), a_parts:DIL04
- BAT1: value 6.25 -> DC 6.25 AC 0
- R2: value 2 -> 1000000; device a_parts:0204V -> a_parts:R0402
- moved R2 12.7 mm to (-61.0, -267.9)
Connections:
- removed net N$2: R7.1, R8.1, R9.2
- new net FB: R2.1, R7.1, R8.1, R9.2, U1.1
- new net VOUT: LED1.A, R8.2, U1.4
- net GND: now also U1.2
- net LED-: now also LED1.K; no longer R2.2
- net VCC: now also U1.3; no longer R2.1, R8.2
- net VDD: now also R2.2
Changed lines of the file:
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@@
 <attribute name="SPICEPREFIX" value="R" x="-14.5" y="-68.1" size="1.016" layer="27" ratio="12" display="off"/>
 </element>
-<element name="BAT1" library="a_parts" package="BATTCON_9V" value="6.25" x="22.4" y="-169.6" smashed="yes">
+<element name="BAT1" library="a_parts" package="BATTCON_9V" value="DC 6.25 AC 0" x="22.4" y="-169.6" smashed="yes">
 <attribute name="NAME" x="19.86" y="-179.76" size="1.27" layer="25" rot="R90"/>
 <attribute name="SPICEPREFIX" value="V" x="22.4" y="-169.6" size="1.778" layer="27" display="off"/>
@@
 <attribute name="SPICEPREFIX" value="R" x="-38" y="-219.5" size="1.016" layer="27" ratio="12" display="off"/>
 </element>
-<element name="R2" library="a_parts" package="0204V" value="2" x="-49.5" y="-262.6" smashed="yes">
-<attribute name="NAME" x="-51.6336" y="-261.4316" size="1.27" layer="25" ratio="10"/>
-<attribute name="SPICEPREFIX" value="R" x="-49.5" y="-262.6" size="1.778" layer="27" display="off"/>
-<attribute name="VALUE" x="-51.6336" y="-264.9114" size="1.27" layer="27" ratio="10"/>
+<element name="U1" library="a_parts" package="DIL04" value="" x="-55.4" y="-260.7" smashed="yes">
+<attribute name="NAME" x="-58.785" y="-260.7" size="0.8128" layer="25" font="vector" ratio="12" rot="R90" align="bottom-center"/>
+<attribute name="SPICEMODEL" value="VSMOD" x="-55.4" y="-260.7" size="1.778" layer="27" display="off"/>
+<attribute name="SPICEPREFIX" value="S" x="-55.4" y="-260.7" size="1.778" layer="27" display="off"/>
+<attribute name="VALUE" x="-55.4" y="-260.7" size="0.8" layer="27" font="vector" ratio="12" rot="R90" align="center"/>
+</element>
+<element name="LED1" library="a_parts" package="LED3MM" value="LED3MM" x="-57.2" y="-267.6" smashed="yes">
+<attribute name="NAME" x="-55.295" y="-267.219" size="1.27" layer="25" ratio="10"/>
+<attribute name="SPICEMODEL" value="DMOD" x="-57.2" y="-267.6" size="1.778" layer="27" display="off"/>
+<attribute name="SPICEPREFIX" value="D" x="-57.2" y="-267.6" size="1.778" layer="27" display="off"/>
+<attribute name="VALUE" x="-55.295" y="-269.251" size="1.27" layer="27" ratio="10"/>
+</element>
+<element name="R2" library="a_parts" package="R0402" value="1000000" x="-61" y="-267.9" smashed="yes">
+<attribute name="NAME" x="-62.1" y="-267.9" size="0.7" layer="25" font="vector" ratio="10" rot="R90" align="bottom-center"/>
+<attribute name="SPICEPREFIX" value="R" x="-61" y="-267.9" size="0.8" layer="27" ratio="12" display="off"/>
 </element>
 </elements>
@@
 <contactref element="U3" pad="5"/>
 <contactref element="BAT1" pad="+"/>
-<contactref element="R8" pad="2"/>
-<contactref element="R2" pad="1"/>
-<wire x1="-50.77" y1="-262.6" x2="-34.4" y2="-219.5" width="0" layer="19" extent="1-1"/>
-<wire x1="22.4" y1="-169.6" x2="-34.4" y2="-219.5" width="0" layer="19" extent="1-1"/>
+<contactref element="U1" pad="3"/>
+<wire x1="-54.13" y1="-256.89" x2="22.4" y2="-169.6" width="0" layer="19" extent="1-1"/>
 <wire x1="10.9" y1="2.35" x2="22.4" y2="-169.6" width="0" layer="19" extent="1-1"/>
 </signal>
@@
 <contactref element="BAT2" pad="-"/>
 <contactref element="R9" pad="1"/>
+<contactref element="U1" pad="2"/>
 <wire x1="22.4" y1="-182.554" x2="22.4" y2="-212.854" width="0" layer="19" extent="1-1"/>
 <wire x1="-38.5" y1="-219.5" x2="22.4" y2="-212.854" width="0" layer="19" extent="1-1"/>
+<wire x1="-54.13" y1="-264.51" x2="-38.5" y2="-219.5" width="0" layer="19" extent="1-1"/>
 <wire x1="15" y1="1.7" x2="22.4" y2="-182.554" width="0" layer="19" extent="1-1"/>
 <wire x1="13.1" y1="3" x2="15" y2="1.7" width="0" layer="19" extent="1-1"/>
@@
 <contactref element="U3" pad="1"/>
 <contactref element="R1" pad="2"/>
-<contactref element="R2" pad="2"/>
-<wire x1="13.1" y1="2.35" x2="-48.23" y2="-262.6" width="0" layer="19" extent="1-1"/>
+<contactref element="LED1" pad="K"/>
+<wire x1="13.1" y1="2.35" x2="-55.93" y2="-267.6" width="0" layer="19" extent="1-1"/>
 <wire x1="15" y1="3.3" x2="13.1" y2="2.35" width="0" layer="19" extent="1-1"/>
 </signal>
@@
 <contactref element="R5" pad="2"/>
 <contactref element="BAT2" pad="+"/>
+<contactref element="R2" pad="2"/>
+<wire x1="-60.5" y1="-267.9" x2="22.4" y2="-199.9" width="0" layer="19" extent="1-1"/>
 <wire x1="28.9" y1="13.1" x2="22.4" y2="-199.9" width="0" layer="19" extent="1-1"/>
 </signal>
-<signal name="N$2">
+<signal name="FB">
 <contactref element="R7" pad="1"/>
 <contactref element="R8" pad="1"/>
 <contactref element="R9" pad="2"/>
+<contactref element="U1" pad="1"/>
+<contactref element="R2" pad="1"/>
 <wire x1="-37.5" y1="-219.5" x2="-35.4" y2="-219.5" width="0" layer="19" extent="1-1"/>
+<wire x1="-56.67" y1="-264.51" x2="-37.5" y2="-219.5" width="0" layer="19" extent="1-1"/>
+<wire x1="-61.5" y1="-267.9" x2="-56.67" y2="-264.51" width="0" layer="19" extent="1-1"/>
 <wire x1="-15" y1="-68.1" x2="-35.4" y2="-219.5" width="0" layer="19" extent="1-1"/>
 </signal>
+<signal name="VOUT">
+<contactref element="R8" pad="2"/>
+<contactref element="U1" pad="4"/>
+<contactref element="LED1" pad="A"/>
+<wire x1="-56.67" y1="-256.89" x2="-34.4" y2="-219.5" width="0" layer="19" extent="1-1"/>
+<wire x1="-58.47" y1="-267.6" x2="-56.67" y2="-256.89" width="0" layer="19" extent="1-1"/>
+</signal>
 </signals>
