File: mp28164/mp28164-buck-boost-flashlight-driver-tester-mk-1.0.2.opamp.only.brd (EAGLE design)
At the start: 20 x 20 mm, 13 parts, among them U3 OPA333

Commit message: whole bunch of crap in here
Parts:
- removed BAT1: 6.25, a_parts:BATTCON_9V
- removed BAT2: DC 2.5 AC 0, a_parts:BATTCON_9V
- removed U3: OPA333, a_parts:SC70
- added LED1: LED3MM, a_parts:LED3MM
- R2: value 2 -> 1; device a_parts:0204V -> a_parts:R0402
- R3: value 75000 -> 15000
- R7: value 10000 -> 1
- moved R2 265.2 mm to (1.50, -2.40)
- moved R9 239.3 mm to (2.90, 16.2), turned to 90 degrees
- moved R6 237.1 mm to (11.6, 13.6), turned to 90 degrees
- moved R8 234.4 mm to (15.7, 9.35), turned to 90 degrees
- moved R7 87.0 mm to (15.1, 13.8), turned to 90 degrees
- moved R3 84.6 mm to (8.70, 13.8), turned to 90 degrees
- moved R5 20.6 mm to (9.00, 16.3)
- moved C5 15.6 mm to (5.80, 14.3), turned to 90 degrees
Connections:
- removed net N$2: R7.1, R8.1, R9.2
- removed net VCC: BAT1.+, R2.1, R8.2, U3.5
- new net FB: R2.1, R8.1, R9.2
- new net LED+: LED1.A
- new net VOUT: R8.2
- new net VSWITCH: R2.2
- net GND: now also R6.1; no longer BAT1.-, BAT2.-, U3.2
- net LED-: now also LED1.K; no longer R2.2, U3.1
- net OPAMP-: no longer R6.1, U3.3
- net OPAMP_OUT: no longer R7.2, U3.4
- net VDD: no longer BAT2.+
Routing:
- removed copper zone on layer 1, net GND
- removed copper zone on layer 16, net GND
Other:
- board text removed: ">VERSION"
- board text removed: "TPS63020 Buck-Boost LED Driver"
