File: mp28164/mp28164-buck-boost-flashlight-driver-tester-mk-1.0.2.opamp.only.sch (EAGLE design)
At the start: 13 parts, among them U3 OPA333

Commit message: whole bunch of crap in here
Parts:
- removed BAT1: 6.25, a_parts:BATTERY9V
- removed BAT2: DC 2.5 AC 0, a_parts:BATTERY9V
- removed U3: OPA333, a_parts:OPAMPOPA333-SC-70
- added LED1: LED3MM, a_parts:LED3MM
- added S1: V_SWITCH, ngspice-simulation:V_SWITCH
- added V1: DC 6V AC 0, ngspice-simulation:VOLTAGE
- added V2: DC 2.5V AC 0, ngspice-simulation:VOLTAGE
- added X1: OPAMP, ngspice-simulation:OPAMP
- R2: value 2 -> 1; device a_parts:RESISTOR0204/2V -> a_parts:RESISTORR0402
- R3: value 75000 -> 15000
- R7: value 10000 -> 1
Connections:
- removed net N$2: R7.1, R8.1, R9.2
- removed net VCC: BAT1.+, R2.1, R8.2, U3.V+
- new net FB: R2.1, R8.1, R9.2
- new net LED+: LED1.A, S1.NM
- new net VOUT: R8.2, S1.NP, V1.+
- new net VSWITCH: R2.2, S1.NCP
- net GND: now also R6.1, S1.NCM, V1.-, V2.-, X1.VSS; no longer BAT1.-, BAT2.-, U3.V-
- net LED-: now also LED1.C, X1.P; no longer R2.2, U3.IN+
- net OPAMP-: now also X1.N; no longer R6.1, U3.IN-
- net OPAMP_OUT: now also X1.VOUT; no longer R7.2, U3.OUT
- net VDD: now also V2.+, X1.VDD; no longer BAT2.+
Other:
- moved on the sheet: R1, R2, R6, R7, R8, R9
