File: mp28164/mp28164-buck-boost-flashlight-driver-tester-mk-1.0.5.opamp.only.brd (EAGLE design)
At the start: 20 x 20 mm, 13 parts, among them U3 OPA333

Commit message: whole bunch of crap in here
Parts:
- removed BAT1: 6.25, a_parts:BATTCON_9V
- removed BAT2: DC 2.5 AC 0, a_parts:BATTCON_9V
- removed C5: .0000000068, a_parts:C0402
- removed R2: 2, a_parts:0204V
- removed R3: 75000, a_parts:R0402
- removed R5: 1000, a_parts:R0402
- removed R6: 100000, a_parts:R0402
- removed R7: 10000, a_parts:R0402
- removed R8: 750000, a_parts:R0402
- removed U3: OPA333, a_parts:SC70
- added C14: 0.000001, a_parts:C0402
- added C8: .000000001, a_parts:C0402
- added LED1: LED3MM, a_parts:LED3MM
- added R11: 15K, a_parts:R0402
- added R12: 47000, a_parts:R0402
- added R13: 75K, a_parts:R0402
- added R14: 360000, a_parts:R0402
- added S1: VSMOD, a_parts:DIL04
- R10: value 1000 -> 10000
- R9: value 68000 -> 10000
- moved R9 240.4 mm to (9.00, 16.3), turned to 180 degrees
- renumbered R4 to R10
Connections:
- removed net N$2: R7.1, R8.1, R9.2
- removed net VDD: BAT2.+, R5.2
- new net FB: R11.2, R12.1, R13.1, S1.1
- new net PWM: R9.2
- new net VOUT: LED1.A, R13.2, S1.4
- net GND: now also C14.2, R11.1, S1.2; no longer BAT1.-, BAT2.-, C5.2, R9.1, U3.2
- net LED-: now also LED1.K; no longer R2.2, U3.1
- net LOWPASS: now also C14.1, R14.2, R9.1; no longer C5.1, R5.1, R6.2
- net OPAMP-: now also C8.1, R14.1; no longer R3.2, R6.1, U3.3
- net OPAMP_OUT: now also C8.2, R12.2; no longer R3.1, R7.2, U3.4
- net VCC: now also S1.3; no longer BAT1.+, R2.1, R8.2, U3.5
Routing:
- removed copper zone on layer 1, net GND
- removed copper zone on layer 16, net GND
Other:
- board text removed: ">VERSION"
- board text removed: "TPS63020 Buck-Boost LED Driver"
