File: mp28164/mp28164-buck-boost-flashlight-driver-tester-mk-1.1.0.sch (EAGLE design)
At the start: 30 parts, among them J1 AVR_SPI_PRG_6PTH, U1 MPS28164, U2 ATTINY25-20MU, U3 OPA399, U4 V_REG_ENTLV700

Commit message: whole bunch of crap in here
Parts:
- removed C2: 10uF, a_parts:CAPACITOR-CERAMICC0805-TIGHTER
- removed C3: 22uF, a_parts:CAPACITOR-CERAMICC0805-TIGHTER
- added FB, LP, OA_NEG, OA_OUT: M01SMD-1MM-DIA-NS, a_parts:M01SMD-1MM-DIA-NS
- C1, C4: device a_parts:CAPACITOR-CERAMICC0805-TIGHTER -> a_parts:CAPACITOR-CERAMICC1206
- L1: device a_parts:INDUCTORXAR7030 -> a_parts:INDUCTORXAL7070
- R1: device a_parts:RESISTORR0805-TIGHTER -> a_parts:RESISTORR1206
- R4: value 4.7k -> 1k
- R5: value 360k -> 1M; device a_parts:RESISTORR0402 -> a_parts:TRIMPOTEVM3Y-LESS
- R6: value 1k -> 10k; device a_parts:RESISTORR0402 -> a_parts:TRIMPOTEVM3Y-LESS
- R7: value 75k -> 100k; device a_parts:RESISTORR0402 -> a_parts:TRIMPOTEVM3Y-LESS
- R8: value 1k -> 100k; device a_parts:RESISTORR0402 -> a_parts:TRIMPOTEVM3Y-LESS
- R9: value 750k -> 1M; device a_parts:RESISTORR0402 -> a_parts:TRIMPOTEVM3Y-LESS
- U2: value ATTINY25-20MU -> ATTINY1310M1; device a_parts:ATTINY45TINY85-20-QFN -> a_parts:ATTINY1310M1
Connections:
- removed net N$1: C6.1, R5.2, R6.2
- new net LOWPASS: C6.1, LP.1, R5.CCW, R6.WIPER
- net ALTPWM/MOSI: now also R6.CCW; no longer R6.1
- net FB: now also FB.1, R8.CCW, R9.WIPER; no longer R8.2, R9.2
- net GND: no longer C2.2, C3.2
- net OPAMP-: now also OA_NEG.1, R5.WIPER, R7.WIPER; no longer R5.1, R7.1
- net OPAMP_OUT: now also OA_OUT.1, R7.CW, R8.WIPER; no longer R7.2, R8.1
- net VBAT: no longer C2.1
- net VOUT: now also R9.CW; no longer C3.1, R9.1
Other:
- note removed: "0.5V R1 = ---------- Gain * Iout"
- note removed: "Gain = 25 (INA190A1) Iout = 1.5A R1 = 13 mOhm"
- moved on the sheet: C6, R10, U2
