File: mp28164/opamp-tester-mk-1.0.0.sch (EAGLE design)
At the start: 30 parts, among them J1 AVR_SPI_PRG_6PTH, U1 MPS28164, U2 ATTINY25-20MU, U3 OPA399, U4 V_REG_ENTLV700

Commit message: whole bunch of crap in here
Parts:
- removed +, -, IN+, IN-: M01PTH-1MM-CIR-NS, a_parts:M01PTH-1MM-CIR-NS
- removed C6: 6800pF, a_parts:CAPACITOR-CERAMICC0402
- removed C7, C8: 1uF, a_parts:CAPACITOR-CERAMICC0402
- removed L1: 2.2uH, a_parts:INDUCTORXAR7030
- removed R2: 19.1K, a_parts:RESISTORR0402
- removed R3: 4.7K, a_parts:RESISTORR0402
- removed U4: V_REG_ENTLV700, a_parts:V_REG_ENTLV700
- added FB, LED+, LP, OA-, OA>: M01PTH-0.7MM-CIR, a_parts:M01PTH-0.7MM-CIR
- added LED: M03SCREW, a_parts:M03SCREW
- added PWR: M02PTH-2MM, a_parts:M02PTH-2MM
- C1, C2: value 10uF -> 1uF; device a_parts:CAPACITOR-CERAMICC0805-TIGHTER -> a_parts:CAPACITOR-CERAMICC0402
- C3: value 22uF -> 1uF; device a_parts:CAPACITOR-CERAMICC0805-TIGHTER -> a_parts:CAPACITOR-CERAMICC0402
- C4: value 22uF -> 1000pF; device a_parts:CAPACITOR-CERAMICC0805-TIGHTER -> a_parts:CAPACITOR-CERAMICC0402
- C5: value 100nF -> 6800pF
- J1: value AVR_SPI_PRG_6PTH -> AVR_SPI_PRG_6SMD_TEST_POINTS; device a_parts:AVR_SPI_PRG_6PTH -> a_parts:AVR_SPI_PRG_6SMD_TEST_POINTS
- R1: device a_parts:RESISTORR0805-TIGHTER -> a_parts:RESISTORR1206
- R10: value 68k -> 15k
- R4: value 4.7k -> 10k
- R5: value 360k -> 1M; device a_parts:RESISTORR0402 -> a_parts:TRIMPOTEVM3Y-LESS
- R6: value 1k -> 10k; device a_parts:RESISTORR0402 -> a_parts:TRIMPOTEVM3Y-LESS
- R7: value 75k -> 100k; device a_parts:RESISTORR0402 -> a_parts:TRIMPOTEVM3Y-LESS
- R8: value 1k -> 100k; device a_parts:RESISTORR0402 -> a_parts:TRIMPOTEVM3Y-LESS
- R9: value 750k -> 100k; device a_parts:RESISTORR0402 -> a_parts:TRIMPOTEVM3Y-LESS
- U1: value MPS28164 -> OPA399; device a_parts:MPS28164 -> a_parts:OPAMPOPA333-SC-70
- U2: value ATTINY25-20MU -> ATTINY1310M1; device a_parts:ATTINY45TINY85-20-QFN -> a_parts:ATTINY1310M1
- U3: value OPA399 -> V_REG_ENTLV700; device a_parts:OPAMPOPA333-SC-70 -> a_parts:V_REG_ENTLV700
Connections:
- removed net L1: L1.1, U1.SW1
- removed net L2: L1.2, U1.SW2
- removed net N$1: C6.1, R5.2, R6.2
- removed net VDD: C5.2, U1.VCC
- removed net VOUT: +.1, C3.1, C4.1, R9.1, U1.VOUT
- new net LED+: LED+.1, LED.3, R9.CW
- new net LOWPASS: C5.1, LP.1, R5.CW, R6.WIPER
- net ALTPWM/MOSI: no longer R6.1
- net FB: now also FB.1, R8.CW, R9.WIPER; no longer R8.2, R9.2, U1.FB
- net GND: now also C1.1, C2.1, C3.1, C4.1, C5.2, LED.1, PWR.1, U1.V-, U3.GND; no longer C1.2, C2.2, C3.2, C4.2, C5.1, C6.2, C7.1, C8.1, IN-.1, R3.1, U1.AGND, U1.PGND, U3.V-, U4.GND
- net LED-: now also LED.2, U1.IN+; no longer -.1, U3.IN+
- net OPAMP-: now also OA-.1, R5.WIPER, R7.WIPER, U1.IN-; no longer R5.1, R7.1, U3.IN-
- net OPAMP_OUT: now also C4.2, OA>.1, R7.CCW, R8.WIPER, U1.OUT; no longer R7.2, R8.1, U3.OUT
- net PWM/MISO: now also R6.CCW; no longer U1.MODE/SYNC
- net VBAT: now also PWR.2; no longer C1.1, C2.1, IN+.1, U1.EN, U1.VIN
- net VBAT_RECT: now also U3.EN, U3.IN; no longer R2.1, U4.EN, U4.IN
- net VCC: now also C1.2, C2.2, C3.2, U1.V+, U3.OUT; no longer C7.2, C8.2, U3.V+, U4.OUT
- net VDIV/SCK: no longer R2.2, R3.2
Other:
- note added: "???"
- note removed: "0.5V R1 = ---------- Gain * Iout"
- note removed: "Gain = 25 (INA190A1) Iout = 1.5A R1 = 13 mOhm"
- moved on the sheet: C1, C2, C3, C4, C5, R1, R10, U2
