File: mp28164/mp28164-buck-boost-flashlight-driver-tester-mk-2.0.2.sch (EAGLE design)
At the start: 28 parts, among them J1 AVR_SPI_PRG_6PTH, U1 MPS28164, U2 ATTINY25-20MU, U3 INA190RSW, U4 TLV30028DCK

Commit message: wip buck boost
Parts:
- removed JP2: M021X02_NO_SILK, a_parts:M021X02_NO_SILK
- added +, -: M01PTH-1.2MM-NS, a_parts:M01PTH-1.2MM-NS
- FRAME1: VERSION v2.1 -> v1.2
- JP1: value M021X02_NO_SILK -> M02PTH-CENTERED; device a_parts:M021X02_NO_SILK -> a_parts:M02PTH-CENTERED
- U2: value ATTINY25-20MU -> ATTINY1310M1; device a_parts:ATTINY45TINY85-20-QFN -> a_parts:ATTINY1310M1
Connections:
- net GND: now also -.1; no longer JP2.1
- net LED+: now also +.1; no longer JP2.2
Other:
- note removed: "For 1.8V operation, U2 = ATTINY{2,4,8}5-10MU U4 = TLV70018DCK"
- note removed: "For 2.8V operation, U2 = ATTINY{2,4,8}5-20MU U4 = TLV70028DCK"
- moved on the sheet: U2
