File: mp3431/mp3431-led-boost-driver-17mm-mk-1.0.0.sch (EAGLE design)
At the start: 34 parts, among them J1 AVR_SPI_PRG_6SMD-1.27MM, U1 MP3431, U2 INA190RSW, U3 V_REG_ENTLV700, U4 ATTINY45TINY85-20-QFN

Commit message: more mp3431 wip
Parts:
- removed C10: ???, a_parts:CAPACITOR-CERAMICC0402
- removed R10: ???, a_parts:RESISTORR0402
- removed R9: 20k, a_parts:RESISTORR0402
- removed VIN+, VIN-: M01PTH-1.2MM-NS, a_parts:M01PTH-1.2MM-NS
- added C12, C14, C16: 1uF, a_parts:CAPACITOR-CERAMICC0402
- added C15: 1nF, a_parts:CAPACITOR-CERAMICC0402
- C2: value 4.7uF -> 68uF; device a_parts:CAPACITOR-CERAMICC0402 -> a_parts:CAPACITOR-CERAMICC1206
- C3, C4: value 47uF -> 4.7uF; device a_parts:CAPACITOR-CERAMICC1206 -> a_parts:CAPACITOR-CERAMICC0402
- C5: value 1uF -> 22nF
- C7: value 1nF -> ???
- C8: value 1uF -> 47uF; device a_parts:CAPACITOR-CERAMICC0402 -> a_parts:CAPACITOR-CERAMICC1206
- C9: value 22nF -> 47uF; device a_parts:CAPACITOR-CERAMICC0402 -> a_parts:CAPACITOR-CERAMICC1206
- L1: value 1uH -> 1.5uH; device a_parts:INDUCTORXAL7070 -> a_parts:INDUCTORXAR7030
- LED+, LED-: value M01PTH-1.2MM-NS -> M01SMD-1.6MMX3.2MM; device a_parts:M01PTH-1.2MM-NS -> a_parts:M01SMD-1.6MMX3.2MM
- R8: value 130k -> ???
Connections:
- net COMP: now also C7.2; no longer C10.2
- net COMP_MID: now also C7.1, R8.2; no longer C10.1, R10.2
- net GND: now also C12.1, C14.1, C15.1, C16.2, C2.2, C3.2, C8.1, R8.1; no longer C2.1, C3.1, C7.1, C8.2, R10.1, R9.1, VIN-.1
- net MODE_PD: no longer R8.2, R9.2
- net PWM/MISO: now also C15.2; no longer C7.2
- net SOFTSTART: now also C5.2; no longer C9.2
- net VBAT: now also C2.1, C3.1; no longer VIN+.1
- net VCC: now also C12.2, C14.2, C16.1; no longer C5.2, C8.1
- net VDD: now also C4.2; no longer C2.2, R8.1
- net VOUT: now also C8.2, C9.2; no longer C3.2, C4.2
Other:
- moved on the sheet: C1, C2, C3, C4, C5, C6, C7, C8, C9, D1, ENABLE, L1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
