File: mp3431/mp3431-boost-tester-mk-1.0.0.sch (EAGLE design)
At the start: 34 parts, among them J1 AVR_SPI_PRG_6SMD-1.27MM, U1 MP3431, U2 INA190RSW, U3 V_REG_ENTLV700, U4 ATTINY45TINY85-20-QFN

Commit message: wip buck boost
Parts:
- FRAME1: VERSION v2.0.1 -> v1.0
Changed lines of the file:
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@@
 <part name="FRAME1" library="a_parts" deviceset="FRAME-LETTER" device="NO_PACKAGE">
 <attribute name="DESIGNER" value="sean@yak.net"/>
-<attribute name="VERSION" value="v2.0.1"/>
+<attribute name="VERSION" value="v1.0"/>
 </part>
 <part name="SUPPLY2" library="a_parts" deviceset="VCC" device=""/>
