File: mp3431/mp3431-boost-tester-mk-2.0.0.brd (EAGLE design)
At the start: 20 x 17.5 mm, 34 parts, among them J1 AVR_SPI_PRG_6SMD-1.27MM, U1 MP3431, U2 INA190RSW, U3 V_REG_ENTLV700, U4 ATTINY45TINY85-20-QFN

Commit message: wip buck boost
Connections:
- net GND: no longer LED-.P$1
- net VBAT: now also LED-.P$1
Routing:
- net LED+: track 18.6 -> 17.6 mm
- net VCC: track 22.3 -> 22.9 mm
Other:
- board text added: "Buck-Boost (return to VIN)"
- board text added: "MP3431"
- board text removed: "MP3431 Boost (return to GND)"
