File: mp3431/mp3431-boost-tester-mk-2.0.0.sch (EAGLE design)
At the start: 28 parts, among them J1 AVR_SPI_PRG_6PTH, U1 MPS28164, U2 ATTINY25-20MU, U3 INA190RSW, U4 TLV30028DCK

Commit message: wip buck boost
Parts:
- removed EN: JUMPER-PAD-2-NOYES_SILK, a_parts:JUMPER-PAD-2-NOYES_SILK
- removed JP1, JP2: M021X02_NO_SILK, a_parts:M021X02_NO_SILK
- added C10: ???, a_parts:CAPACITOR-CERAMICC0402
- added C7: 1nF, a_parts:CAPACITOR-CERAMICC0402
- added C8: 1uF, a_parts:CAPACITOR-CERAMICC0402
- added C9: 22nF, a_parts:CAPACITOR-CERAMICC0402
- added ENABLE: (no value), a_parts:JUMPER-PAD-3-NOSMALL_BOX_SILK
- added LED+, LED-, VIN+, VIN-: M01PTH-1.2MM-NS, a_parts:M01PTH-1.2MM-NS
- C1: value 22uF -> 68uF
- C2: value 100nF -> 4.7uF
- C4: value 1uF -> 47uF; device a_parts:CAPACITOR-CERAMICC0402 -> a_parts:CAPACITOR-CERAMICC1206
- C6: value 10nF -> 0.1uF
- FRAME1: VERSION v2.1 -> v2.0
- J1: value AVR_SPI_PRG_6PTH -> AVR_SPI_PRG_6SMD-1.27MM; device a_parts:AVR_SPI_PRG_6PTH -> a_parts:AVR_SPI_PRG_6SMD-1.27MM
- L1: device a_parts:INDUCTORXAL60XX -> a_parts:INDUCTORXAL7070
- MODE: value JUMPER-PAD-2-NOYES_SILK -> (none); device a_parts:JUMPER-PAD-2-NOYES_SILK -> a_parts:JUMPER-PAD-3-NOSMALL_BOX_SILK
- R10: value DNP -> ???
- R4: value 1.02K -> 6.8k
- R5: value 220R -> 1k
- R6: value 0R -> 75K
- R7: value 560K -> 15K
- R8: value 100K -> 130k
- R9: value DNP -> 20k
- U1: value MPS28164 -> MP3431; device a_parts:MPS28164 -> a_parts:MP3431
- U2: value ATTINY25-20MU -> INA190RSW; device a_parts:ATTINY45TINY85-20-QFN -> a_parts:INA190RSW
- U3: value INA190RSW -> V_REG_ENTLV700; device a_parts:INA190RSW -> a_parts:V_REG_ENTLV700
- U4: value TLV30028DCK -> ATTINY45TINY85-20-QFN; device a_parts:V_REG_ENTLV700XXDCR -> a_parts:ATTINY45TINY85-20-QFN
Connections:
- removed net EN: EN.2, R9.2, U1.EN
- removed net L1: L1.1, U1.SW1
- removed net L2: L1.2, U1.SW2
- removed net MODE/SYNC: MODE.2, R10.2, U1.MODE/SYNC
- new net BST: C6.2, U1.BST
- new net COMP: C10.2, U1.COMP
- new net COMP_MID: C10.1, R10.2
- new net ENABLE: ENABLE.2, U1.EN
- new net MODE: MODE.2, U1.MODE
- new net MODE_PD: MODE.3, R8.2, R9.2
- new net SOFTSTART: C9.2, U1.SS
- new net SW: C6.1, L1.2, U1.SW
- net ALTPWM/MOSI: now also ENABLE.3, U4.PB0(MOSI); no longer EN.1, MODE.1, U2.PB0(MOSI)
- net CSOUT: now also R5.1, U2.OUT; no longer R6.2, U3.OUT
- net FB: now also R5.2, R6.2; no longer R6.1, R8.2
- net GND: now also C2.1, C3.1, C4.1, C7.1, C8.2, C9.1, R10.1, R7.1, R9.1, U1.ILM, VIN-.1; no longer C2.2, C3.2, C4.2, C6.2, JP1.1, JP2.1, R5.2, R8.1
- net LED+: now also LED+.1, R6.1, U2.VIN-; no longer JP2.2, R7.1, U3.VIN-
- net PWM/MISO: now also C7.2, U4.PB1(MISO); no longer U2.PB1(MISO)
- net REF: now also U2.REF; no longer C6.1, R5.1, U3.REF
- net RST: now also U4.RESET; no longer U2.RESET
- net VBAT: now also ENABLE.1, L1.1, LED-.1, MODE.1, VIN+.1; no longer JP1.2, R10.1, R9.1
- net VBAT_RECT: now also U3.EN, U3.IN; no longer U4.EN, U4.IN
- net VCC: now also C8.1, U2.EN, U3.OUT, U4.VCC; no longer C4.1, U3.EN, U3.VCC, U4.OUT
- net VDD: now also C2.2, R8.1, U1.VDD; no longer C2.1, U1.VCC
- net VDIV/SCK: now also U4.PB2(SCK/ADC1); no longer U2.PB2(SCK/ADC1)
- net VOUT: now also C3.2, C4.2, U2.VIN+; no longer C3.1, U3.VIN+
Other:
- note removed: "For 1.8V operation, U2 = ATTINY{2,4,8}5-10MU U4 = TLV70018DCK"
- note removed: "For 2.8V operation, U2 = ATTINY{2,4,8}5-20MU U4 = TLV70028DCK"
- moved on the sheet: C1, C2, C3, C4, C5, C6, D1, J1, L1, R1, R10, R2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
