File: tps610891/tps610891-boost-to-vin-flashlight-driver-tester-mk-1.0.0.brd (EAGLE design)
At the start: 17.6 x 17.6 mm, 23 parts, among them J1 AVR_SPI_PRG_6SMD-1.27MM, U1 MPS28164, U3 INA190RSW, U4 V_REG_ENTLV700, U5 ATTINY45TINY85-20-QFN

Commit message: wip buck boost
Parts:
- removed +, -: M01SMD-1.6MMX3.2MM-NS, a_parts:1X01-SMD-1.6MMX3.2MM-NS
- removed U5: ATTINY45TINY85-20-QFN, a_parts:QFN20
- added C6: TBD, a_parts:C0402
- added C8: 1uF, a_parts:C0402
- added C9: 10nF, a_parts:C0402
- added JP1, JP2: M021X02_NO_SILK, a_parts:1X02_NO_SILK
- added R10, R8: 100K, a_parts:R0402
- added R11: TBD, a_parts:R0402
- added R9: 68K, a_parts:R0402
- added U2: ATTINY25-20MU, a_parts:QFN20
- C2: value 100nF -> 47uF; device a_parts:C0402 -> a_parts:C1206
- C3: value 47uF -> 1uF; device a_parts:C1206 -> a_parts:C0402
- C4: value 1uF -> 0.1uF
- C5: value 1uF -> TBD
- C7: value 1nF -> 1uF
- J1: value AVR_SPI_PRG_6SMD-1.27MM -> AVR_SPI_PRG_6PTH; device a_parts:2X3-1.27MM-SMD -> a_parts:2X3
- L1: device a_parts:XAL7070 -> a_parts:XAL60XX
- R4: value 6.8k -> 1.02K
- R5: value 6.8k -> 220R
- R6: value 75K -> 0R
- R7: value 15K -> 560K
- U1: value MPS28164 -> TPS610891; device a_parts:MPS28164 -> a_parts:VQFN-11
- U4: value V_REG_ENTLV700 -> TLV30028DCK
- moved C5 23.1 mm to (-11.4, -2.80), flipped to the top
- moved C4 20.2 mm to (-2.10, -2.80), flipped to the top
- moved J1 12.4 mm to (17.0, 4.50), flipped to the top, turned to 90 degrees
- moved C7 9.00 mm to (12.6, 3.50), flipped to the top, turned to 180 degrees
- moved R2 8.50 mm to (9.50, 14.0), turned to 0 degrees
- moved C3 7.57 mm to (4.50, 4.00), turned to 0 degrees
- moved R3 7.52 mm to (12.0, 14.0), turned to 180 degrees
- moved R5 7.26 mm to (11.5, 9.60), turned to 90 degrees
- moved U4 7.16 mm to (11.0, 12.0), turned to 270 degrees
- moved D1 5.83 mm to (8.50, 11.0), turned to 90 degrees
- moved R1 5.15 mm to (10.0, 5.50), turned to 270 degrees
- moved U1 4.50 mm to (4.50, 6.20), turned to 0 degrees
- moved L1 4.50 mm to (4.50, 11.5), turned to 180 degrees
- moved C1 3.54 mm to (1.50, 5.50), turned to 270 degrees
- moved U3 3.52 mm to (12.5, 5.30), flipped to the top, turned to 180 degrees
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Connections:
- removed net L1: L1.P$1, U1.10
- removed net L2: L1.P$2, U1.8
- new net BOOT: C4.2, U1.10
- new net COMP: C6.1, R11.1, U1.4
- new net FSW: R9.2, U1.1
- new net ILIM: R10.1, U1.8
- new net N$1: C4.1, L1.P$1, R9.1, U1.11@1, U1.11@2, U1.11@3
- new net N$5: C5.1, R11.2
- net ALTPWM/MOSI: now also U1.7, U2.11; no longer U1.2, U5.11
- net CSOUT: now also R6.2; no longer R5.2
- net FB: now also R6.1, R7.2, R8.2, U1.3; no longer R5.1, R6.2, R7.1, U1.6
- net GND: now also C5.2, C6.2, C7.2, C8.1, C9.2, JP1.1, R10.2, R5.2, R8.1, U2.8, U2.PAD; no longer -.P$1, C4.2, C5.1, C7.1, R7.2, U1.9, U5.8, U5.PAD
- net LED+: now also JP2.2, R7.1; no longer +.P$1, R6.1
- net PWM/MISO: now also U2.12; no longer C7.2, U5.12
- net REF: now also C9.1, R5.1
- net RST: now also U2.1; no longer U5.1
- net VBAT: now also JP1.2, JP2.1, L1.P$2, U1.9; no longer U1.1, U1.11@1, U1.11@2
- net VCC: now also C7.1, C8.2, U2.15; no longer C4.1, C5.2, U5.15
- net VDD: now also C3.1, U1.2; no longer C2.1, U1.4
- net VDIV/SCK: now also U2.14; no longer U5.14
- net VOUT: now also C2.1, U1.6; no longer C3.1, U1.7@1, U1.7@2
Routing:
- net VCC: track 24.4 -> 0.00 mm, vias 5 -> 0
- net ALTPWM/MOSI: track 23.1 -> 0.00 mm, vias 1 -> 0
- net VDIV/SCK: track 15.7 -> 0.00 mm, vias 2 -> 0
- net RST: track 13.6 -> 0.00 mm, vias 2 -> 0
- net PWM/MISO: track 13.3 -> 0.00 mm
- net LED+: track 12.1 -> 0.00 mm, vias 1 -> 0
- net FB: track 8.68 -> 0.00 mm, vias 1 -> 0
- net CSOUT: track 8.58 -> 0.00 mm, vias 1 -> 0
- net VBAT_RECT: track 5.87 -> 0.00 mm
- net REF: track 5.28 -> 0.00 mm
- net VBAT: track 3.77 -> 0.00 mm, vias 9 -> 0
- net VDD: track 3.41 -> 0.00 mm
- net VOUT: track 2.90 -> 0.00 mm, vias 1 -> 0
- removed copper zone on layer 1, net L1
- removed copper zone on layer 1, net L2
- removed copper zone on layer 1, net VBAT
- removed copper zone on layer 16, net VBAT
- removed copper zone on layer 1, net VOUT
Other:
- board size 17.6 x 17.6 mm -> 20 x 15 mm
- board text added: "+"
- board text added: "-"
- board text added: "IN"
- board text added: "MP28614 LED Driver Test Board"
- board text added: "OUT"
- board text removed: "LED Driver"
- board text removed: "MP28614"
